File: NSE2022/Eagle/PCB/testESP ver.1/testESP ver.1.sch (EAGLE design)
At the start: 2 parts, among them CN1 DM3AT

Commit message: Update testESP ver.1.sch
Parts:
- removed CN1: DM3AT, microSD:DM3AT
- added 3-REG1: (no value), Chip 3-Terminal Regulator:AZ1117CH-3.3TRG1
- added C1, C2: 22uf, rcl:C-EUC0603
- added L1: OSXX1608C1A, ChipLED:OSXX1608C1A
- added R1: 2k, rcl:R-US_R0201
- added R2, R3: 10k, rcl:R-US_R0201
- added T1, T2: (no value), ChipTransister:NPN_SS8050-G
- added TVC1, TVC2, TVC3: (no value), TVC Diode:ESD5484FCT5G
- added U$2, U$3: TS-06104, Switches:TS-06104
- added U$4, U$5: 19_2.54, JumperPins:19_2.54
- added U1: CP2102N-A01-GQFN28, CP2102N-A01-GQFN28:CP2102N-A01-GQFN28
- added USB1: (no value), USB:MICRO-B_ZX62R-B-5P
Connections:
- new net +3V3: 3-REG1.2_OUTPUT, 3-REG1.VOUT, C1.1
- new net +5V: 3-REG1.3_INPUT, C2.1, R1.2
- new net +D: TVC3.2_AN, USB1.3_D+
- new net -D: TVC2.2_AN, USB1.2_D-
- new net DCD: U1.DCD
- new net DTR: R3.1, T2.2
- new net EN: T1.3
- new net GND: 3-REG1.1_GND, C1.2, C2.2, L1.CT, TVC1.1_CT, TVC2.1_CT, TVC3.1_CT, USB1.5_GND
- new net IO0: T2.3
- new net N$1: L1.AN, R1.1
- new net N$2: R3.2, T1.1
- new net N$3: U1.RXD
- new net N$4: U1.TXD
- new net N$5: R2.2, T2.1
- new net N$6: U1.RTS
- new net N$7: U1.CTS
- new net RI: U1.RI/CLK
- new net RTS: R2.1, T1.2
- new net VBUS: TVC1.2_AN, USB1.1_VBUS(5V)
Other:
- note added: "SS8050-G"
- moved on the sheet: U$1
