File: NSE2022/Eagle/PCB/ESP devkit ver.1/ESP devkit ver.1.sch (EAGLE design)
At the start: 19 parts, among them U1 CP2102N-A01-GQFN28

Commit message: a
Parts:
- removed U$2, U$3: TS-06104, Switches:TS-06104
- added C3, C4, C6, C7: 0.1uF, rcl:C-EUC0603
- added C5: 4.7uF, rcl:C-EUC0402
- added C8: 22uF, rcl:C-EUC0603
- added EN, IO0: TS-06104, Switches:TS-06104
- added R4: 2k, rcl:R-US_R0201
- added R5: 10k, rcl:R-US_R0201
- added R6: 22k, rcl:R-US_R0201
- added R7: 47k, rcl:R-US_R0201
Connections:
- net N$7 renamed CTS
- removed net N$3: U1.RXD
- removed net N$6: U1.RTS
- new net CLK: U$1.20_CLK, U$5.P$1
- new net CMD: U$1.19_CMD, U$4.P$18
- new net CPVBUS: R6.2, R7.2, U1.VBUS
- new net DSR: U1.DSR
- new net IO12: U$1.14_IO12, U$4.P$13
- new net IO13: U$1.16_IO13, U$4.P$15
- new net IO14: U$1.13_IO14, U$4.P$12
- new net IO15: U$1.23_IO15, U$5.P$4
- new net IO16: U$1.27_IO16_NC, U$5.P$8
- new net IO17: U$1.28_IO17_NC, U$5.P$9
- new net IO18: U$1.30_IO18, U$5.P$11
- new net IO19: U$1.31_IO19, U$5.P$12
- new net IO2: U$1.24_IO2, U$5.P$5
- new net IO21: U$1.33_IO21, U$5.P$14
- new net IO22: U$1.36_IO22, U$5.P$17
- new net IO23: U$1.37_IO23, U$5.P$18
- new net IO25: U$1.10_IO25, U$4.P$9
- new net IO26: U$1.11_IO26, U$4.P$10
- new net IO27: U$1.12_IO27, U$4.P$11
- new net IO32: U$1.8_IO32, U$4.P$7
- new net IO33: U$1.9_IO33, U$4.P$8
- new net IO34: U$1.6_IO34, U$4.P$5
- new net IO35: U$1.7_IO35, U$4.P$6
- new net IO4: U$1.26_IO4, U$5.P$7
- new net IO5: U$1.29_IO5, U$5.P$10
- new net N$10: R5.1, U1.!SUSPENDB
- new net N$8: R4.2, U1.!RST
- new net NC: U$1.32_NC
- new net RXD: U$1.35_TXD0, U$5.P$16, U1.RXD
- new net SD0: U$1.21_SD0, U$5.P$2
- new net SD1: U$1.22_SD1, U$5.P$3
- new net SD2: U$1.17_SD2, U$4.P$16
- new net SD3: U$1.18_SD3, U$4.P$17
- new net S_VN: U$1.5_SENSOR_VN, U$4.P$4
- new net S_VP: U$1.4_SENSOR_VP, U$4.P$3
- new net TXD: U$1.34_RXD0, U$5.P$15, U1.TXD
- net +3V3: now also C5.1, C6.1, C7.1, C8.1, R4.1, U$1.2_VDD33, U$4.P$1, U1.VDD, U1.VREGIN
- net +5V: now also U$4.P$19
- net +D: now also U1.D+
- net -D: now also U1.D-
- net EN: now also C4.1, EN.D, U$1.3_EN, U$4.P$2
- net GND: now also C3.2, C4.2, C5.2, C6.2, C7.2, C8.2, EN.B, IO0.B, R5.2, R7.1, U$1.15_GND, U$1.1_GND, U$1.38_GND, U$1.39_GND, U$4.P$14, U$5.P$13, U$5.P$19, U1.GND
- net IO0: now also C3.1, IO0.D, U$1.25_IO0, U$5.P$6
- net N$4: now also U1.DTR; no longer U1.TXD
- net RTS: now also U1.RTS
- net VBUS: now also R6.1
Other:
- moved on the sheet: 3-REG1, C1, C2, L1, R1, R2, R3, T1, T2, TVC1, TVC2, TVC3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
