File: NSE2022/Eagle/PCB/cansat_test ver.2/cansat.sch (EAGLE design)
At the start: 80 parts, among them U2 CP2102N-A01-GQFN28

Commit message: a
Parts:
- renumbered U$1 to ESP_LED1, U$2 to ESP_LED2, U$3 to IMCHECK, U$4 to RAS_LED1, U$5 to RAS_LED2, U$6 to RAS_LED3
Connections:
- removed net +5V2: C1.+
- removed net GND2: C1.-, C21.-, C22.-, C6.-, DCDC1.GND
- net +5V: now also C1.+
- net GND: now also C1.-, C21.-, C22.-, C6.-, DCDC1.GND
Other:
- moved on the sheet: R19, R20
