File: NSE2022/Eagle/PCB/Rotally Encoder_ver1.0/Rotall Encoder ver1.0.brd (EAGLE design)
At the start: 16.5 x 14.7 mm, 6 parts, among them U1 AS5600

Commit message: a
Parts:
- added C10, C11, C12, C13, C14, C15, C16, C17, C18, C19, C20, C21, C22, C23, C24, C3, C4, C5, C6, C7, C8, C9: (no value), rcl:C0603
- added JP1, JP10, JP11, JP12, JP2, JP4, JP5, JP6, JP7, JP8, JP9: 06X01, PinHeader:06X01
- added R10, R11, R12, R13, R14, R15, R16, R17, R18, R19, R20, R21, R22, R23, R24, R3, R4, R5, R6, R7, R8, R9: (no value), rcl:R0603
- added U10, U11, U12, U2, U3, U4, U5, U6, U7, U8, U9: AS5600, AS5600:AS5600
- moved C1 2.82 mm to (0.89, 4.06)
- moved JP3 2.82 mm to (6.48, 1.52)
- moved C2 2.82 mm to (4.70, 4.06)
- moved R1 2.82 mm to (8.51, 4.06)
- moved R2 2.82 mm to (12.3, 4.06)
- moved U1 2.82 mm to (6.35, 8.76)
Connections:
- net +3V3: now also C10.1, C12.1, C14.1, C16.1, C18.1, C20.1, C22.1, C24.1, C4.1, C6.1, C8.1, JP1.2, JP10.2, JP11.2, JP12.2, JP2.2, JP4.2, JP5.2, JP6.2, JP7.2, JP8.2, JP9.2, U10.VDD3V3, U11.VDD3V3, U12.VDD3V3, U2.VDD3V3, U3.VDD3V3, U4.VDD3V3, U5.VDD3V3, U6.VDD3V3, U7.VDD3V3, U8.VDD3V3, U9.VDD3V3
- net +5V: now also C11.1, C13.1, C15.1, C17.1, C19.1, C21.1, C23.1, C3.1, C5.1, C7.1, C9.1, JP1.1, JP10.1, JP11.1, JP12.1, JP2.1, JP4.1, JP5.1, JP6.1, JP7.1, JP8.1, JP9.1, R10.2, R11.2, R12.2, R13.2, R14.2, R15.2, R16.2, R17.2, R18.2, R19.2, R20.2, R21.2, R22.2, R23.2, R24.2, R3.2, R4.2, R5.2, R6.2, R7.2, R8.2, R9.2, U10.VDD5V, U11.VDD5V, U12.VDD5V, U2.VDD5V, U3.VDD5V, U4.VDD5V, U5.VDD5V, U6.VDD5V, U7.VDD5V, U8.VDD5V, U9.VDD5V
- net GND: now also C10.2, C11.2, C12.2, C13.2, C14.2, C15.2, C16.2, C17.2, C18.2, C19.2, C20.2, C21.2, C22.2, C23.2, C24.2, C3.2, C4.2, C5.2, C6.2, C7.2, C8.2, C9.2, JP1.3, JP10.3, JP11.3, JP12.3, JP2.3, JP4.3, JP5.3, JP6.3, JP7.3, JP8.3, JP9.3, U10.DIR, U10.GND, U11.DIR, U11.GND, U12.DIR, U12.GND, U2.DIR, U2.GND, U3.DIR, U3.GND, U4.DIR, U4.GND, U5.DIR, U5.GND, U6.DIR, U6.GND, U7.DIR, U7.GND, U8.DIR, U8.GND, U9.DIR, U9.GND
- net OUT: now also JP1.6, JP10.6, JP11.6, JP12.6, JP2.6, JP4.6, JP5.6, JP6.6, JP7.6, JP8.6, JP9.6, U10.OUT, U11.OUT, U12.OUT, U2.OUT, U3.OUT, U4.OUT, U5.OUT, U6.OUT, U7.OUT, U8.OUT, U9.OUT
- net SCL: now also JP1.4, JP10.4, JP11.4, JP12.4, JP2.4, JP4.4, JP5.4, JP6.4, JP7.4, JP8.4, JP9.4, R11.1, R13.1, R15.1, R17.1, R19.1, R21.1, R23.1, R3.1, R5.1, R7.1, R9.1, U10.SCL, U11.SCL, U12.SCL, U2.SCL, U3.SCL, U4.SCL, U5.SCL, U6.SCL, U7.SCL, U8.SCL, U9.SCL
- net SDA: now also JP1.5, JP10.5, JP11.5, JP12.5, JP2.5, JP4.5, JP5.5, JP6.5, JP7.5, JP8.5, JP9.5, R10.1, R12.1, R14.1, R16.1, R18.1, R20.1, R22.1, R24.1, R4.1, R6.1, R8.1, U10.SDA, U11.SDA, U12.SDA, U2.SDA, U3.SDA, U4.SDA, U5.SDA, U6.SDA, U7.SDA, U8.SDA, U9.SDA
Routing:
- net +5V: track 47.3 -> 364.3 mm
- net OUT: track 17.6 -> 198.5 mm, vias 0 -> 5
- net GND: track 21.9 -> 201.5 mm, vias 1 -> 0
- net +3V3: track 9.60 -> 175.7 mm
- net SDA: track 8.21 -> 157.3 mm
- net SCL: track 8.63 -> 124.7 mm
Other:
- board size 16.5 x 14.7 mm -> 80 x 49.5 mm
