File: NSE2022/Eagle/PCB/NSE2022 Electro_ESPtest ver.1/NSE2022 Electro_ESPtest ver.1.brd (EAGLE design)
At the start: 87.6 x 83.8 mm, 59 parts, among them CN1 DM3AT, U1 CP2102N-A01-GQFN28

Commit message: a
Parts:
- added U$2: (no value), logo:LOGO
- 3-REG1: value (none) -> 5-3.3
- CON1: value (none) -> FP
- CON2: value (none) -> BATT
- CON3: value (none) -> SV1
- CON4: value (none) -> SV2
- CON5: value (none) -> SV3
- CON6: value (none) -> SV4
- DCDC1: value (none) -> 12-5
- JP1, JP3: value (none) -> 19pin
- JP2: value (none) -> 7pin
- moved 3-REG1 1.53 mm to (36.4, 6.60)
- moved R7 1.02 mm to (26.7, 11.0)
- moved C2 0.80 mm to (30.6, 9.91)
- moved L1 0.80 mm to (31.2, 7.49)
- moved R1 0.80 mm to (30.2, 7.49)
- moved C1 0.80 mm to (30.6, 12.4)
- moved R6 0.51 mm to (26.7, 9.78)
- turned SW3 to 0 degrees
Connections:
- removed net IO14: JP1.12
- removed net IO15: JP3.4
- removed net IO16: JP3.8
- removed net IO17: JP3.9
- removed net IO18: JP3.11
- removed net IO19: JP3.12
- removed net IO2: JP3.5
- removed net IO21: JP3.14
- removed net IO22: JP3.17
- removed net IO23: JP3.18
- removed net IO25: JP1.9
- removed net IO26: JP1.10
- removed net IO27: JP1.11
- removed net IO32: JP1.7
- removed net IO33: JP1.8
- removed net IO5: JP3.10
- removed net N$6: 3-REG1.1_GND, C1.2, C2.2, L1.CT
- net FP_CHECKER: now also JP1.7
- net GND: now also 3-REG1.1_GND, C1.2, C2.2, L1.CT
- net GPSRX: now also JP3.5
- net GPSTX: now also JP3.4
- net IMBUSY: now also JP1.12
- net IMRX: now also JP3.8
- net IMTX: now also JP3.9
- net MISO: now also JP3.12
- net MOSI: now also JP3.18
- net SCK: now also JP3.11
- net SCL: now also JP3.17
- net SDA: now also JP3.14
- net SS: now also JP3.10
- net SV1: now also JP1.11
- net SV2: now also JP1.10
- net SV3: now also JP1.9
- net SV4: now also JP1.8
Routing:
- net GND: track 0.00 -> 452.0 mm, vias 0 -> 11
- net +3V3: track 0.00 -> 280.9 mm, vias 0 -> 9
- net +5V: track 0.00 -> 215.2 mm, vias 0 -> 4
- net IMTX: track 0.00 -> 189.4 mm, vias 0 -> 3
- net SS: track 0.00 -> 187.0 mm, vias 0 -> 5
- net MOSI: track 0.00 -> 184.8 mm, vias 0 -> 5
- net IMRX: track 0.00 -> 169.4 mm, vias 0 -> 4
- net MISO: track 0.00 -> 140.1 mm, vias 0 -> 6
- net IMBUSY: track 0.00 -> 137.4 mm, vias 0 -> 3
- net CLK: track 0.00 -> 130.6 mm, vias 0 -> 4
- net GPSRX: track 0.00 -> 127.5 mm, vias 0 -> 3
- net GPSTX: track 0.00 -> 121.7 mm, vias 0 -> 3
- net SCK: track 0.00 -> 115.1 mm, vias 0 -> 6
- net IO4: track 0.00 -> 114.1 mm, vias 0 -> 2
- net FP_CHECKER: track 0.00 -> 110.9 mm
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- added copper zone on layer 1, net GND
- added copper zone on layer 16, net GND
Other:
- board text added: "3V3"
- board text added: "3v3"
- board text added: "5V"
- board text added: "CLK"
- board text added: "CMD"
- board text added: "CTS"
- board text added: "DTR"
- board text added: "EN"
- board text added: "FC"
- board text added: "GND"
- board text added: "GPSRX"
- board text added: "GPSTX"
- board text added: "IMB"
- board text added: "IMRX"
- board text added: "IMTX"
- board text added: "IO0"
- board text added: "IO12"
- board text added: "IO13"
- board text added: "IO34"
- board text added: "IO35"
- board text added: "IO4"
- board text added: "MISO"
- board text added: "MOSI"
- board text added: "RTS"
- board text added: "RXD"
- board text added: "SCK"
- board text added: "SCL"
- board text added: "SD0"
- board text added: "SD1"
- board text added: "SD2"
- board text added: "SD3"
- board text added: "SDA"
- board text added: "SS"
- board text added: "SV1"
- board text added: "SV2"
- board text added: "SV3"
- board text added: "SV4"
- board text added: "SVN"
- board text added: "SVP"
- board text added: "TXD"

Commit message: a
Routing:
- net MOSI: track 184.8 -> 119.7 mm, vias 5 -> 3
- net IMRX: track 169.4 -> 115.7 mm
- net MISO: track 140.1 -> 87.6 mm
- net IMTX: track 189.4 -> 139.0 mm, vias 3 -> 5
- net IO4: track 114.1 -> 64.0 mm, vias 2 -> 4
- net SS: track 187.0 -> 137.2 mm, vias 5 -> 4
- net SCL: track 110.6 -> 159.1 mm, vias 3 -> 1
- net +3V3: track 280.9 -> 233.7 mm
- net SCK: track 115.1 -> 161.8 mm, vias 6 -> 2
- net GND: track 452.0 -> 491.6 mm, vias 11 -> 6
- net S_VP: track 90.6 -> 66.9 mm, vias 3 -> 1
- net RXD: track 89.0 -> 68.4 mm, vias 1 -> 3
- net DTR: track 38.2 -> 54.7 mm, vias 2 -> 1
- net SD0: track 108.0 -> 124.3 mm, vias 2 -> 0
- net SV3: track 95.4 -> 111.5 mm, vias 3 -> 5
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