File: NSE2022/Eagle/PCB/NSE2022 Electro_ESPtest ver.1/NSE2022 Electro_ESPtest ver.1.sch (EAGLE design)
At the start: 59 parts, among them CN1 DM3AT, U1 CP2102N-A01-GQFN28

Commit message: a
Parts:
- 3-REG1: value (none) -> 5-3.3
- CON1: value (none) -> FP
- CON2: value (none) -> BATT
- CON3: value (none) -> SV1
- CON4: value (none) -> SV2
- CON5: value (none) -> SV3
- CON6: value (none) -> SV4
- DCDC1: value (none) -> 12-5
- JP1, JP3: value (none) -> 19pin
- JP2: value (none) -> 7pin
Connections:
- removed net IO14: JP1.12
- removed net IO15: JP3.4
- removed net IO16: JP3.8
- removed net IO17: JP3.9
- removed net IO18: JP3.11
- removed net IO19: JP3.12
- removed net IO2: JP3.5
- removed net IO21: JP3.14
- removed net IO22: JP3.17
- removed net IO23: JP3.18
- removed net IO25: JP1.9
- removed net IO26: JP1.10
- removed net IO27: JP1.11
- removed net IO32: JP1.7
- removed net IO33: JP1.8
- removed net IO5: JP3.10
- removed net N$6: 3-REG1.1_GND, C1.2, C2.2, L1.CT
- net FP_CHECKER: now also JP1.7
- net GND: now also 3-REG1.1_GND, C1.2, C2.2, L1.CT
- net GPSRX: now also JP3.5
- net GPSTX: now also JP3.4
- net IMBUSY: now also JP1.12
- net IMRX: now also JP3.8
- net IMTX: now also JP3.9
- net MISO: now also JP3.12
- net MOSI: now also JP3.18
- net SCK: now also JP3.11
- net SCL: now also JP3.17
- net SDA: now also JP3.14
- net SS: now also JP3.10
- net SV1: now also JP1.11
- net SV2: now also JP1.10
- net SV3: now also JP1.9
- net SV4: now also JP1.8
