File: NSE2022/Eagle/PCB/NSE2022 Electro_ESPtest ver.1 - コピー/NSE2022 Electro_ESPtest ver.1.brd (EAGLE design)
At the start: 90 x 85 mm, 60 parts, among them CN1 DM3AT, CON1 FP, CON2 BATT, CON3 SV1, CON4 SV2, CON5 SV3, CON6 SV4, U1 CP2102N-A01-GQFN28

Commit message: kato_ESP
Parts:
- moved IM1 150.9 mm to (-75.9, 29.5)
- moved JP2 130.2 mm to (-115.8, -6.70)
- moved R15 130.2 mm to (-110.0, -4.16)
- moved R16 130.2 mm to (-112.6, -9.24)
- moved R5 118.6 mm to (-81.8, -18.7)
- moved U2 116.6 mm to (-54.9, -11.4), turned to 180 degrees
- moved R4 116.1 mm to (-79.8, -17.7)
- moved C9 115.7 mm to (-52.8, 14.9)
- moved USB1 114.7 mm to (-86.7, -7.92), turned to 270 degrees
- moved 3-REG1 114.5 mm to (-74.6, -21.4), turned to 90 degrees
- moved R1 113.8 mm to (-80.8, -17.5)
- moved R6 113.8 mm to (-84.3, -15.2)
- moved R7 113.8 mm to (-84.3, -14.0)
- moved TVC1 113.8 mm to (-84.3, -16.6)
- moved TVC2 113.8 mm to (-84.3, -17.6)
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Routing:
- net GND: track 452.0 -> 0.00 mm, vias 11 -> 0
- net +3V3: track 280.9 -> 0.00 mm, vias 9 -> 0
- net +5V: track 215.2 -> 0.00 mm, vias 4 -> 0
- net IMTX: track 189.4 -> 0.00 mm, vias 3 -> 0
- net SS: track 187.0 -> 0.00 mm, vias 5 -> 0
- net MOSI: track 184.8 -> 0.00 mm, vias 5 -> 0
- net IMRX: track 169.4 -> 0.00 mm, vias 4 -> 0
- net MISO: track 140.1 -> 0.00 mm, vias 6 -> 0
- net IMBUSY: track 137.4 -> 0.00 mm, vias 3 -> 0
- net CLK: track 130.6 -> 0.00 mm, vias 4 -> 0
- net GPSRX: track 127.5 -> 0.00 mm, vias 3 -> 0
- net GPSTX: track 121.7 -> 0.00 mm, vias 3 -> 0
- net SCK: track 115.1 -> 0.00 mm, vias 6 -> 0
- net IO4: track 114.1 -> 0.00 mm, vias 2 -> 0
- net FP_CHECKER: track 110.9 -> 0.00 mm
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Other:
- board size 90 x 85 mm -> 85 x 85 mm
