File: NSE2022/Eagle/PCB/runback_ver1/cansat.sch (EAGLE design)
At the start: 83 parts, among them U2 CP2102N-A01-GQFN28

Commit message: sadasd
Parts:
- removed 3-REG2: (no value), Chip 3-Terminal Regulator:AZ1117CH-3.3TRG1
- removed C1: 22uF, rcl:C-EUC0603
- removed C12, C13, C14, C15: 4.7uF, rcl:CPOL-EUE2.5-7
- removed C2, C3, C6, C7, C8: 0.1uF, rcl:C-EUC0603
- removed C4, C5: 22uf, rcl:C-EUC0603
- removed C9: 4.7uF, rcl:C-EUC0402
- removed CON4, CON5: (no value), Connector:2.5_MINI-SPOX_4PIN
- removed DCDC1: 5-3.3, DC-DC:3.3V0.5A_M78AR05-0.5
- removed EN1, IO1: TS-06104, Switches:TS-06104
- removed ESP32_WROOM32D: ESP32-WROOM-32D, ESP32:ESP32-WROOM-32D
- removed JP2: 7pin, JumperPins:7_2.54
- removed PW: OSXX1608C1A, ChipLED:OSXX1608C1A
- removed R10, R11: 3.3kR, rcl:R-US_R0603
- removed R12, R13, R14, R21, R7: 10k, rcl:R-US_R0201
- removed R15, R20: 2k, rcl:R-US_R0201
- removed R16, R17: 100k, rcl:R-EU_0207/10
- removed R18: 22k, rcl:R-US_R0201
- removed R19: 47k, rcl:R-US_R0201
- removed R8, R9: 2.2kR, rcl:R-US_R0603
- removed T3, T4: (no value), ChipTransister:NPN_SS8050-G
- removed TVC4, TVC5, TVC6: (no value), TVC Diode:ESD5484FCT5G
- removed U2: CP2102N-A01-GQFN28, CP2102N-A01-GQFN28:CP2102N-A01-GQFN28
- removed USB2: (no value), USB:MICRO-B_ZX62R-B-5P
- added U$2: ESP32, ESP32_dev:ESP32
Connections:
- removed net +D: TVC6.2_AN, U2.D+, USB2.3_D+
- removed net -D: TVC5.2_AN, U2.D-, USB2.2_D-
- removed net AS_SCL: CON4.4, CON5.4, PIN_R.P$3, R8.2
- removed net AS_SDA: CON4.3, CON5.3, PIN_R.P$6, R9.2
- removed net CLK: ESP32_WROOM32D.20_CLK, PIN_R.P$19
- removed net CMD: ESP32_WROOM32D.19_CMD, PIN_L.P$18
- removed net CPVBUS: R18.2, R19.2, U2.VBUS
- removed net DTR: JP2.P$7, R13.1, R17.2, T4.2, U2.DTR
- removed net N$13: PW.AN, R15.1
- removed net N$14: R13.2, T3.1
- removed net N$15: R14.2, T4.1
- removed net N$16: R20.2, U2.!RST
- removed net N$17: R21.1, U2.!SUSPENDB
- removed net N$7: ESP32_WROOM32D.36_IO22, R10.2, R8.1
- removed net N$8: ESP32_WROOM32D.33_IO21, R11.2, R9.1
- removed net RTS: JP2.P$1, R14.1, R16.2, T3.2, U2.RTS
- removed net SD0: ESP32_WROOM32D.21_SD0, PIN_R.P$18
- removed net SD1: ESP32_WROOM32D.22_SD1, PIN_R.P$17
- removed net SD2: ESP32_WROOM32D.17_SD2, PIN_L.P$16
- removed net SD3: ESP32_WROOM32D.18_SD3, PIN_L.P$17
- new net IO10: PIN_L.P$17, U$2.GPIO10
- new net IO11: PIN_L.P$18, U$2.GPIO11
- new net IO6: PIN_R.P$19, U$2.GPIO6
- new net IO7: PIN_R.P$18, U$2.GPIO7
- new net IO8: PIN_R.P$17, U$2.GPIO8
- new net IO9: PIN_L.P$16, U$2.GPIO9
- new net SCL: PIN_R.P$3, U$2.GPIO22
- new net SDA: PIN_R.P$6, U$2.GPIO21
- net +3V3: now also U$2.3.3V; no longer 3-REG2.2_OUTPUT, 3-REG2.VOUT, C1.1, C15.+, C2.1, C5.1, C8.1, C9.1, DCDC1.VOUT, ESP32_WROOM32D.2_3V3, JP2.P$4, R12.2, R20.1, R7.2, U2.VDD, U2.VREGIN
- net +5V: now also U$2.5V; no longer 3-REG2.3_INPUT, C12.+, C13.+, C14.+, C4.1, CON4.2, CON5.2, DCDC1.VIN, R15.2, R18.1, TVC4.2_AN, USB2.1_VBUS(5V)
- net EN: now also U$2.EN; no longer C3.1, C7.1, EN1.D, ESP32_WROOM32D.3_EN, R12.1, T3.3
- net GND: now also U$2.GND1, U$2.GND2, U$2.GND3; no longer 3-REG2.1_GND, C1.2, C12.-, C13.-, C14.-, C15.-, C2.2, C3.2, C4.2, C5.2, C6.2, C7.2, C8.2, C9.2, CON4.1, CON5.1, DCDC1.GND, EN1.B, ESP32_WROOM32D.15_GND, ESP32_WROOM32D.1_GND, ESP32_WROOM32D.32_NC, ESP32_WROOM32D.38_GND, ESP32_WROOM32D.39_GND, IO1.B, JP2.P$2, PW.CT, R10.1, R11.1, R16.1, R17.1, R19.1, R21.2, TVC4.1_CT, TVC5.1_CT, TVC6.1_CT, U2.GND, USB2.5_GND
- net IM_BUSY: now also U$2.GPIO14; no longer ESP32_WROOM32D.13_IO14
- net IM_RESET: now also U$2.GPIO12; no longer ESP32_WROOM32D.14_IO12
- net IM_RX: now also PIN_R.P$15, RASPBERRYPI_4B.GPIO1, U$2.GPIO2; no longer ESP32_WROOM32D.28_IO17, PIN_R.P$11
- net IM_TX: now also PIN_R.P$16, RASPBERRYPI_4B.GPIO0, U$2.GPIO15; no longer ESP32_WROOM32D.27_IO16, PIN_R.P$12
- net IO13: now also U$2.GPIO13; no longer ESP32_WROOM32D.16_IO13
- net IO27: now also U$2.GPIO27; no longer ESP32_WROOM32D.12_IO27
- net IO5: now also U$2.GPIO5; no longer ESP32_WROOM32D.29_IO5
- net LED1: now also U$2.GPIO34; no longer ESP32_WROOM32D.6_IO34
- net LED2: now also U$2.GPIO35; no longer ESP32_WROOM32D.7_IO35
- net MD_LB: now also U$2.GPIO26; no longer ESP32_WROOM32D.11_IO26
- net MD_LF: now also U$2.GPIO25; no longer ESP32_WROOM32D.10_IO25
- net MD_RB: now also U$2.GPIO0; no longer C6.1, ESP32_WROOM32D.25_IO0, IO1.D, T4.3
- net MD_RF: now also U$2.GPIO4; no longer ESP32_WROOM32D.26_IO4
- net RP_MISO: now also U$2.GPIO19; no longer ESP32_WROOM32D.31_IO19
- net RP_MOSI: now also U$2.GPIO23; no longer ESP32_WROOM32D.37_IO23, R7.1
- net RP_RX: now also PIN_R.P$11, U$2.GPIO17; no longer ESP32_WROOM32D.24_IO2, PIN_R.P$15, RASPBERRYPI_4B.GPIO1
- net RP_SCK: now also U$2.GPIO18; no longer ESP32_WROOM32D.30_IO18
- net RP_SS: now also U$2.GPIO39; no longer ESP32_WROOM32D.5_SENSOR_VN
- net RP_TX: now also PIN_R.P$12, U$2.GPIO16; no longer ESP32_WROOM32D.23_IO15, PIN_R.P$16, RASPBERRYPI_4B.GPIO0
- net RXD: now also U$2.TX; no longer ESP32_WROOM32D.35_TXD0, JP2.P$6, U2.RXD
- net SENSOR_VP: now also U$2.GPIO36; no longer ESP32_WROOM32D.4_SENSOR_VP
- net SERVO1: now also U$2.GPIO32; no longer ESP32_WROOM32D.8_IO32
- net SERVO2: now also U$2.GPIO33; no longer ESP32_WROOM32D.9_IO33
- net TXD: now also U$2.RX; no longer ESP32_WROOM32D.34_RXD0, JP2.P$5, U2.TXD
Other:
- note added: "IM920c"
- note added: "Motor System"
- note added: "To Bottom"
- note added: "To Top"
- note removed: "IM920"
- note removed: "Motor"
- note removed: "Motor Driver"
- note removed: "Rotally Encorder"
- note removed: "SS8050-G"
- note removed: "USB-UART"
- moved on the sheet: C10, C11, C16, C17, C18, C19, C20, ESP_LED1, ESP_LED2, IMCHECK, R1, R2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

Commit message: sadasd
Parts:
- added TM4, TM5: (no value), TerminalBrock:TERMINAL_SLOPED_2PIN
- added TOBOTTOM, TOTOP: (no value), Connector:2.5_MINI-SPOX_4PIN
Connections:
- net +5V: now also TM4.1, TM5.1
- net GND: now also TM4.2, TM5.2
- net MD_LB: now also TOBOTTOM.2, TOTOP.2
- net MD_LF: now also TOBOTTOM.1, TOTOP.1
- net MD_RB: now also TOBOTTOM.4, TOTOP.4
- net MD_RF: now also TOBOTTOM.3, TOTOP.3
Other:
- note added: "ESP32 (TOP)"
- note added: "GPS (TOP)"
- note added: "I2C (TOP)"
- note added: "IM920c (TOP)"
- note added: "LED (TOP)"
- note added: "Motor System (BOTTOM)"
- note added: "Pins (TOP)"
- note added: "Power (BOTTOM)"
- note added: "Raspberry Pi (TOP)"
- note added: "Servo (TOP)"
- note added: "Switching (BOTTOM)"
- note added: "to Bottom (TOP)"
- note added: "to Top (BOTTOM)"
- note removed: "ESP32"
- note removed: "GPS"
- note removed: "I2C"
- note removed: "IM920c"
- note removed: "LED"
- note removed: "Motor System"
- note removed: "Pins"
- note removed: "Power"
- note removed: "Raspberry Pi"
- note removed: "Servo"
- note removed: "Switching"
- note removed: "To Bottom"
- note removed: "To Top"
- moved on the sheet: C10, C11
