File: NSE2022/Eagle/PCB/runback_ver1/ranback_bottom.sch (EAGLE design)
At the start: 44 parts

Commit message: asd
Parts:
- removed BMX1: BMX055, BMX055:BMX055
- removed CON2, CON3: (no value), Connector:2.5_MINI-SPOX_3PIN
- removed ESP_LED1, ESP_LED2, IMCHECK, RAS_LED1, RAS_LED2, RAS_LED3: OSXX1608C1A, ChipLED:OSXX1608C1A
- removed GPS: AE-GYSFDMAXB, AE-GYSFDMAXB:AE-GYSFDMAXB
- removed IM: IM920C, IM920:IM920C
- removed PIN_L, PIN_R: 19_2.54, JumperPins:19_2.54
- removed R1, R2, R3, R4, R5, R6: 1.5k, rcl:R-US_R0603
- removed RASPBERRYPI_4B: (no value), RASPBERRYPI4B:RASPBERRYPI4B
- removed TM5: (no value), TerminalBrock:TERMINAL_SLOPED_2PIN
- removed TOBOTTOM: (no value), Connector:2.5_MINI-SPOX_4PIN
- removed U$2: ESP32, ESP32_dev:ESP32
- removed U$9: GY-BPM280, BMP280:GY-BPM280
Connections:
- removed net +3V3: IM.VCC, PIN_L.P$1, U$2.3.3V, U$9.CSB, U$9.VCC
- removed net BB_SCL: BMX1.SCL, RASPBERRYPI_4B.GPIO3, U$9.SCK
- removed net BB_SDA: BMX1.SDA, RASPBERRYPI_4B.GPIO2, U$9.SDI
- removed net EN: PIN_L.P$2, U$2.EN
- removed net GPS_RX: GPS.RXD, RASPBERRYPI_4B.GPIO14
- removed net GPS_TX: GPS.TXD, RASPBERRYPI_4B.GPIO15
- removed net IM_BUSY: IM.BUSY/IO1, PIN_L.P$12, U$2.GPIO14
- removed net IM_RESET: IM.RESET, PIN_L.P$13, U$2.GPIO12
- removed net IM_RX: IM.RXD/IO6, PIN_R.P$15, RASPBERRYPI_4B.GPIO1, U$2.GPIO2
- removed net IM_TX: IM.TXD/IO7, PIN_R.P$16, RASPBERRYPI_4B.GPIO0, U$2.GPIO15
- removed net IO10: PIN_L.P$17, U$2.GPIO10
- removed net IO11: PIN_L.P$18, U$2.GPIO11
- removed net IO13: PIN_L.P$15, U$2.GPIO13
- removed net IO27: PIN_L.P$11, U$2.GPIO27
- removed net IO5: PIN_R.P$10, U$2.GPIO5
- removed net IO6: PIN_R.P$19, U$2.GPIO6
- removed net IO7: PIN_R.P$18, U$2.GPIO7
- removed net IO8: PIN_R.P$17, U$2.GPIO8
- removed net IO9: PIN_L.P$16, U$2.GPIO9
- removed net LED1: PIN_L.P$5, R1.1, U$2.GPIO34
- removed net LED2: PIN_L.P$6, R2.1, U$2.GPIO35
- removed net LED3: IM.STATUS, R3.1
- removed net LED4: R4.1, RASPBERRYPI_4B.GPIO17
- removed net LED5: R5.1, RASPBERRYPI_4B.GPIO27
- removed net LED6: R6.1, RASPBERRYPI_4B.GPIO22
- removed net N$1: ESP_LED1.AN, R1.2
- removed net N$2: ESP_LED2.AN, R2.2
- removed net N$3: IMCHECK.AN, R3.2
- removed net N$4: R4.2, RAS_LED1.AN
- removed net N$5: R5.2, RAS_LED2.AN
- removed net N$6: R6.2, RAS_LED3.AN
- removed net RP_MISO: PIN_R.P$8, RASPBERRYPI_4B.GPIO9, U$2.GPIO19
- removed net RP_MOSI: PIN_R.P$2, RASPBERRYPI_4B.GPIO10, U$2.GPIO23
- removed net RP_RX: PIN_R.P$11, U$2.GPIO17
- removed net RP_SCK: PIN_R.P$9, RASPBERRYPI_4B.GPIO11, U$2.GPIO18
- removed net RP_SS: PIN_L.P$4, RASPBERRYPI_4B.GPIO8, U$2.GPIO39
- removed net RP_TX: PIN_R.P$12, U$2.GPIO16
- removed net RXD: PIN_R.P$4, U$2.TX
- removed net SCL: PIN_R.P$3, U$2.GPIO22
- removed net SDA: PIN_R.P$6, U$2.GPIO21
- removed net SENSOR_VP: PIN_L.P$3, U$2.GPIO36
- removed net SERVO1: CON2.3, PIN_L.P$7, U$2.GPIO32
- removed net SERVO2: CON3.3, PIN_L.P$8, U$2.GPIO33
- removed net TXD: PIN_R.P$5, U$2.RX
- net +5V: no longer BMX1.VCC, CON2.2, CON3.2, GPS.5V, PIN_L.P$19, RASPBERRYPI_4B.5V_1, TM5.1, U$2.5V
- net GND: no longer BMX1.GND, CON2.1, CON3.1, ESP_LED1.CT, ESP_LED2.CT, GPS.GND, IM.GND, IMCHECK.CT, PIN_L.P$14, PIN_R.P$1, PIN_R.P$7, RASPBERRYPI_4B.GND_1, RASPBERRYPI_4B.GND_2, RASPBERRYPI_4B.GND_3, RASPBERRYPI_4B.GND_4, RASPBERRYPI_4B.GND_5, RASPBERRYPI_4B.GND_6, RASPBERRYPI_4B.GND_7, RASPBERRYPI_4B.GND_8, RAS_LED1.CT, RAS_LED2.CT, RAS_LED3.CT, TM5.2, U$2.GND1, U$2.GND2, U$2.GND3, U$9.GND, U$9.SDO
- net MD_LB: no longer PIN_L.P$10, TOBOTTOM.2, U$2.GPIO26
- net MD_LF: no longer PIN_L.P$9, TOBOTTOM.1, U$2.GPIO25
- net MD_RB: no longer PIN_R.P$14, TOBOTTOM.4, U$2.GPIO0
- net MD_RF: no longer PIN_R.P$13, TOBOTTOM.3, U$2.GPIO4
