File: NSE2022/Eagle/PCB/runback_ver1/ranback_top.brd (EAGLE design)
At the start: 100 x 61.3 mm, 24 parts

Commit message: a
Parts:
- added U$1: (no value), logo:LOGO
Changed lines of the file:
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@@
 <layer number="98" name="Guide" color="6" fill="1" visible="no" active="no"/>
 <layer number="99" name="SpiceOrder" color="5" fill="1" visible="no" active="no"/>
+<layer number="200" name="200bmp" color="1" fill="10" visible="yes" active="yes"/>
 </layers>
 <board>
@@
 <element name="U$2" library="ESP32_dev" package="ESP32" value="ESP32" x="5.08" y="1.27" smashed="yes"/>
 <element name="U$9" library="BMP280" package="GY-BMP280-FOOTPRINT" value="GY-BPM280" x="97.79" y="10.16" smashed="yes" rot="R90"/>
+<element name="U$1" library="logo" package="LOGO" value="" x="83.82" y="43.18" smashed="yes">
+<attribute name="NAME" x="85.09" y="43.18" size="0.6096" layer="21"/>
+</element>
 </elements>
 <signals>
