File: NSE2022/Eagle/PCB/runback_ver1/ranback_bottom.brd (EAGLE design)
At the start: 168 x 88 mm, 20 parts

Commit message: yoro
Parts:
- moved TOTOP 95.3 mm to (26.7, 5.08)
- moved TM4 92.7 mm to (15.2, 7.62)
- moved TM1 87.6 mm to (31.8, 76.2)
- moved C11 86.4 mm to (20.3, 68.6)
- moved U$7 86.4 mm to (-7.62, 17.8)
- moved U$8 85.5 mm to (-0.38, 41.0)
- moved C10 85.1 mm to (-20.3, 68.6)
- moved C16 85.1 mm to (-7.62, 68.6)
- moved C17 85.1 mm to (15.2, 58.4)
- moved C18 85.1 mm to (0.00, 58.4)
- moved C20 85.1 mm to (7.62, 68.6)
- moved R22 85.1 mm to (0.00, 12.7)
- moved U$10 85.1 mm to (7.62, 17.8)
- moved C19 83.8 mm to (-15.2, 58.4)
- moved MD_R 83.8 mm to (12.7, 78.7)
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Routing:
- net GND: track 242.3 -> 0.00 mm, vias 1 -> 0
- net +5V: track 153.0 -> 0.00 mm
- net +12V: track 146.1 -> 0.00 mm
- net MD_LB: track 106.8 -> 0.00 mm
- net MD_LF: track 102.5 -> 0.00 mm
- net MD_RB: track 85.3 -> 0.00 mm
- net MD_RF: track 84.9 -> 0.00 mm, vias 1 -> 0
- net N$18: track 82.8 -> 0.00 mm
- net N$20: track 54.9 -> 0.00 mm
- net OUT_MD_R1: track 25.4 -> 0.00 mm
- net OUT_MD_R2: track 24.7 -> 0.00 mm
- net N$9: track 23.3 -> 0.00 mm
- net OUT_MD_L1: track 20.1 -> 0.00 mm
- net OUT_MD_L2: track 19.6 -> 0.00 mm, vias 1 -> 0
- net A7_1: track 19.3 -> 0.00 mm
Other:
- board size 168 x 88 mm -> 100 x 88 mm
- board text added: "12V"
- board text added: "5V"
- board text added: "GND"
- board text added: "L1"
- board text added: "L2"
- board text added: "LB"
- board text added: "LF"
- board text added: "R1"
- board text added: "R2"
- board text added: "RB"
- board text added: "RF"

Commit message: repair1
Parts:
- added U$1: (no value), logo:LOGO
Routing:
- net GND: track 0.00 -> 212.1 mm
- net +12V: track 0.00 -> 169.1 mm
- net +5V: track 0.00 -> 131.2 mm, vias 0 -> 2
- net MD_LB: track 0.00 -> 97.9 mm, vias 0 -> 1
- net MD_LF: track 0.00 -> 96.0 mm, vias 0 -> 1
- net MD_RF: track 0.00 -> 79.1 mm, vias 0 -> 2
- net MD_RB: track 0.00 -> 78.1 mm
- net N$18: track 0.00 -> 70.4 mm
- net OUT_MD_L2: track 0.00 -> 32.1 mm, vias 0 -> 2
- net A7_1: track 0.00 -> 27.9 mm
- net N$20: track 0.00 -> 27.4 mm
- net OUT_MD_L1: track 0.00 -> 27.2 mm
- net OUT_MD_R1: track 0.00 -> 23.6 mm
- net OUT_MD_R2: track 0.00 -> 20.4 mm, vias 0 -> 2
- net N$9: track 0.00 -> 16.6 mm
- added copper zone on layer 1, net GND
- added copper zone on layer 16, net GND
Other:
- board text added: "BATT"
- board text added: "Left Motor"
- board text added: "Power to Top"
- board text added: "Right Motor"
