File: NSE2022/Eagle/PCB/runback_ver1.1/ranback_top.brd (EAGLE design)
At the start: 100 x 61.3 mm, 25 parts

Commit message: asdf
Connections:
- removed net IO6: PIN_R.19, U$2.GPIO6
- removed net IO7: PIN_R.18, U$2.GPIO7
- new net IO34: PIN_L.5, U$2.GPIO34
- new net IO35: PIN_L.6, U$2.GPIO35
- net +3V3: now also RASPBERRYPI_4B.3V3_1; no longer U$2.3.3V
- net LED1: now also PIN_R.19, U$2.GPIO6; no longer PIN_L.5, U$2.GPIO34
- net LED2: now also PIN_R.18, U$2.GPIO7; no longer PIN_L.6, U$2.GPIO35
Routing:
- net IO34: track 0.00 -> 5.21 mm
- net IO35: track 0.00 -> 5.19 mm
- net IO7: track 4.09 -> 0.00 mm
- net IO6: track 4.06 -> 0.00 mm
- net LED2: track 94.0 -> 92.3 mm
- net LED1: track 110.3 -> 108.6 mm
Changed lines of the file:
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@@
 <grid distance="50" unitdist="mil" unit="mm" style="lines" multiple="1" display="no" altdistance="5" altunitdist="mil" altunit="mm"/>
 <layers>
-<layer number="1" name="Top" color="4" fill="1" visible="yes" active="yes"/>
+<layer number="1" name="Top" color="4" fill="1" visible="no" active="yes"/>
 <layer number="2" name="Route2" color="16" fill="1" visible="no" active="no"/>
 <layer number="3" name="Route3" color="17" fill="1" visible="no" active="no"/>
@@
 <layer number="14" name="Route14" color="22" fill="1" visible="no" active="no"/>
 <layer number="15" name="Route15" color="23" fill="1" visible="no" active="no"/>
-<layer number="16" name="Bottom" color="1" fill="1" visible="yes" active="yes"/>
+<layer number="16" name="Bottom" color="1" fill="1" visible="no" active="yes"/>
 <layer number="17" name="Pads" color="2" fill="1" visible="yes" active="yes"/>
 <layer number="18" name="Vias" color="2" fill="1" visible="yes" active="yes"/>
@@
 <signal name="LED1">
 <contactref element="R1" pad="1"/>
-<contactref element="U$2" pad="GPIO34"/>
-<contactref element="PIN_L" pad="5"/>
 <wire x1="79.75" y1="10.75" x2="80.25" y2="10.25" width="0.1524" layer="1"/>
 <wire x1="79.75" y1="15" x2="79.75" y2="10.75" width="0.1524" layer="1"/>
@@
 <wire x1="6.25" y1="38" x2="5.25" y2="38" width="0.1524" layer="16"/>
 <wire x1="80.25" y1="10.25" x2="80.43" y2="10.16" width="0.1524" layer="1"/>
-<wire x1="6.25" y1="38" x2="6.35" y2="38.1" width="0.1524" layer="16"/>
-<wire x1="6.25" y1="38.25" x2="2.75" y2="41.75" width="0.1524" layer="1"/>
-<wire x1="2.75" y1="41.75" x2="2.54" y2="41.91" width="0.1524" layer="1"/>
-<wire x1="6.25" y1="38.25" x2="6.35" y2="38.1" width="0.1524" layer="1"/>
 <via x="70" y="27.5" extent="1-16" drill="0.2"/>
+<contactref element="U$2" pad="GPIO6"/>
+<contactref element="PIN_R" pad="19"/>
+<wire x1="31.75" y1="2.5" x2="35.5" y2="2.5" width="0.1524" layer="1"/>
+<wire x1="35.5" y1="2.5" x2="35.56" y2="2.54" width="0.1524" layer="1"/>
+<wire x1="35.56" y1="2.54" x2="70" y2="27.5" width="0" layer="19" extent="1-1"/>
+<wire x1="31.52" y1="2.54" x2="31.75" y2="2.5" width="0" layer="19" extent="1-1"/>
 </signal>
 <signal name="LED2">
 <contactref element="R2" pad="1"/>
-<contactref element="U$2" pad="GPIO35"/>
-<contactref element="PIN_L" pad="6"/>
 <wire x1="73.75" y1="11.75" x2="75.25" y2="10.25" width="0.1524" layer="1"/>
 <wire x1="73.75" y1="27.25" x2="73.75" y2="11.75" width="0.1524" layer="1"/>
@@
 <wire x1="6.5" y1="35.5" x2="12.5" y2="29.5" width="0.1524" layer="16"/>
 <wire x1="75.25" y1="10.25" x2="75.35" y2="10.16" width="0.1524" layer="1"/>
-<wire x1="6.5" y1="35.5" x2="6.35" y2="35.56" width="0.1524" layer="16"/>
-<wire x1="6.25" y1="35.75" x2="2.75" y2="39.25" width="0.1524" layer="1"/>
-<wire x1="2.75" y1="39.25" x2="2.54" y2="39.37" width="0.1524" layer="1"/>
-<wire x1="6.25" y1="35.75" x2="6.35" y2="35.56" width="0.1524" layer="1"/>
 <via x="73.75" y="27.25" extent="1-16" drill="0.2"/>
+<contactref element="U$2" pad="GPIO7"/>
+<contactref element="PIN_R" pad="18"/>
+<wire x1="31.75" y1="5" x2="35.5" y2="5" width="0.1524" layer="1"/>
+<wire x1="35.5" y1="5" x2="35.56" y2="5.08" width="0.1524" layer="1"/>
+<wire x1="31.52" y1="5.08" x2="6.5" y2="35.5" width="0" layer="19" extent="16-16"/>
+<wire x1="31.75" y1="5" x2="31.52" y2="5.08" width="0" layer="19" extent="1-1"/>
 </signal>
 <signal name="SERVO1">
@@
 <contactref element="U$9" pad="VCC"/>
 <contactref element="U$9" pad="CSB"/>
-<contactref element="U$2" pad="3.3V"/>
 <contactref element="PIN_L" pad="1"/>
 <wire x1="6.25" y1="48.5" x2="2.75" y2="52" width="0.1524" layer="1"/>
 <wire x1="2.75" y1="52" x2="2.54" y2="52.07" width="0.1524" layer="1"/>
-<wire x1="6.25" y1="48.5" x2="6.35" y2="48.26" width="0.1524" layer="1"/>
 <wire x1="75.5" y1="23.25" x2="75.5" y2="28.25" width="0.1524" layer="1"/>
 <wire x1="77" y1="21.75" x2="75.5" y2="23.25" width="0.1524" layer="16"/>
@@
 <wire x1="78.25" y1="25" x2="78.5" y2="25.25" width="0.1524" layer="16"/>
 <wire x1="78.25" y1="21.75" x2="78.25" y2="25" width="0.1524" layer="16"/>
-<wire x1="6.5" y1="48.25" x2="6.35" y2="48.26" width="0.1524" layer="16"/>
 <via x="75.5" y="23.25" extent="1-16" drill="0.2"/>
+<contactref element="RASPBERRYPI_4B" pad="3V3_1"/>
+<wire x1="6.25" y1="48.5" x2="10.16" y2="52.07" width="0" layer="19" extent="1-1"/>
+<wire x1="6.5" y1="48.25" x2="6.25" y2="48.5" width="0" layer="19" extent="1-16"/>
 </signal>
 <signal name="+5V">
@@
 <wire x1="31.75" y1="7.75" x2="31.52" y2="7.62" width="0.1524" layer="1"/>
 </signal>
-<signal name="IO7">
-<contactref element="U$2" pad="GPIO7"/>
-<contactref element="PIN_R" pad="18"/>
-<wire x1="31.75" y1="5" x2="35.5" y2="5" width="0.1524" layer="1"/>
-<wire x1="35.5" y1="5" x2="35.56" y2="5.08" width="0.1524" layer="1"/>
-<wire x1="31.75" y1="5" x2="31.52" y2="5.08" width="0.1524" layer="1"/>
-</signal>
 <signal name="IO9">
 <contactref element="U$2" pad="GPIO9"/>
@@
 <wire x1="6.25" y1="5.25" x2="6.35" y2="5.08" width="0.1524" layer="1"/>
 </signal>
-<signal name="IO6">
-<contactref element="U$2" pad="GPIO6"/>
-<contactref element="PIN_R" pad="19"/>
-<wire x1="31.75" y1="2.5" x2="35.5" y2="2.5" width="0.1524" layer="1"/>
-<wire x1="35.5" y1="2.5" x2="35.56" y2="2.54" width="0.1524" layer="1"/>
-<wire x1="31.75" y1="2.5" x2="31.52" y2="2.54" width="0.1524" layer="1"/>
-</signal>
 <signal name="N$1">
 <contactref element="R1" pad="2"/>
@@
 <wire x1="56.5" y1="10.25" x2="56.73" y2="10.16" width="0.1524" layer="1"/>
 </signal>
+<signal name="IO34">
+<contactref element="U$2" pad="GPIO34"/>
+<contactref element="PIN_L" pad="5"/>
+<wire x1="6.25" y1="38.25" x2="2.75" y2="41.75" width="0.1524" layer="1"/>
+<wire x1="2.75" y1="41.75" x2="2.54" y2="41.91" width="0.1524" layer="1"/>
+<wire x1="6.25" y1="38.25" x2="6.35" y2="38.1" width="0" layer="19" extent="1-1"/>
+</signal>
+<signal name="IO35">
+<contactref element="U$2" pad="GPIO35"/>
+<contactref element="PIN_L" pad="6"/>
+<wire x1="6.25" y1="35.75" x2="2.75" y2="39.25" width="0.1524" layer="1"/>
+<wire x1="2.75" y1="39.25" x2="2.54" y2="39.37" width="0.1524" layer="1"/>
+<wire x1="6.25" y1="35.75" x2="6.35" y2="35.56" width="0" layer="19" extent="1-1"/>
+</signal>
 </signals>

Commit message: asdfgfdsasdfgfdsasdfgfdsa
Routing:
- net LED2: track 92.3 -> 105.3 mm, vias 1 -> 3
- net LED1: track 108.6 -> 100.4 mm
Changed lines of the file:
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@@
 <grid distance="50" unitdist="mil" unit="mm" style="lines" multiple="1" display="no" altdistance="5" altunitdist="mil" altunit="mm"/>
 <layers>
-<layer number="1" name="Top" color="4" fill="1" visible="no" active="yes"/>
+<layer number="1" name="Top" color="4" fill="1" visible="yes" active="yes"/>
 <layer number="2" name="Route2" color="16" fill="1" visible="no" active="no"/>
 <layer number="3" name="Route3" color="17" fill="1" visible="no" active="no"/>
@@
 <layer number="14" name="Route14" color="22" fill="1" visible="no" active="no"/>
 <layer number="15" name="Route15" color="23" fill="1" visible="no" active="no"/>
-<layer number="16" name="Bottom" color="1" fill="1" visible="no" active="yes"/>
+<layer number="16" name="Bottom" color="1" fill="1" visible="yes" active="yes"/>
 <layer number="17" name="Pads" color="2" fill="1" visible="yes" active="yes"/>
 <layer number="18" name="Vias" color="2" fill="1" visible="yes" active="yes"/>
@@
 <signal name="LED1">
 <contactref element="R1" pad="1"/>
-<wire x1="79.75" y1="10.75" x2="80.25" y2="10.25" width="0.1524" layer="1"/>
-<wire x1="79.75" y1="15" x2="79.75" y2="10.75" width="0.1524" layer="1"/>
-<wire x1="80.5" y1="15.75" x2="79.75" y2="15" width="0.1524" layer="1"/>
-<wire x1="80.5" y1="28.75" x2="80.5" y2="15.75" width="0.1524" layer="1"/>
-<wire x1="79.5" y1="29.75" x2="80.5" y2="28.75" width="0.1524" layer="1"/>
-<wire x1="70" y1="29.75" x2="79.5" y2="29.75" width="0.1524" layer="1"/>
-<wire x1="70" y1="27.5" x2="70" y2="29.75" width="0.1524" layer="1"/>
-<wire x1="69.5" y1="27" x2="70" y2="27.5" width="0.1524" layer="16"/>
-<wire x1="14.25" y1="27" x2="69.5" y2="27" width="0.1524" layer="16"/>
-<wire x1="6.75" y1="34.5" x2="14.25" y2="27" width="0.1524" layer="16"/>
-<wire x1="5.5" y1="34.5" x2="6.75" y2="34.5" width="0.1524" layer="16"/>
-<wire x1="5.25" y1="34.75" x2="5.5" y2="34.5" width="0.1524" layer="16"/>
-<wire x1="5.25" y1="38" x2="5.25" y2="34.75" width="0.1524" layer="16"/>
-<wire x1="6.25" y1="38" x2="5.25" y2="38" width="0.1524" layer="16"/>
-<wire x1="80.25" y1="10.25" x2="80.43" y2="10.16" width="0.1524" layer="1"/>
-<via x="70" y="27.5" extent="1-16" drill="0.2"/>
 <contactref element="U$2" pad="GPIO6"/>
 <contactref element="PIN_R" pad="19"/>
-<wire x1="31.75" y1="2.5" x2="35.5" y2="2.5" width="0.1524" layer="1"/>
+<wire x1="32" y1="2.5" x2="35.5" y2="2.5" width="0.1524" layer="1"/>
 <wire x1="35.5" y1="2.5" x2="35.56" y2="2.54" width="0.1524" layer="1"/>
-<wire x1="35.56" y1="2.54" x2="70" y2="27.5" width="0" layer="19" extent="1-1"/>
-<wire x1="31.52" y1="2.54" x2="31.75" y2="2.5" width="0" layer="19" extent="1-1"/>
+<wire x1="80.5" y1="11.5" x2="80.5" y2="10.5" width="0.1524" layer="1"/>
+<wire x1="84" y1="15" x2="80.5" y2="11.5" width="0.1524" layer="16"/>
+<wire x1="98" y1="15" x2="84" y2="15" width="0.1524" layer="16"/>
+<wire x1="99" y1="14" x2="98" y2="15" width="0.1524" layer="16"/>
+<wire x1="99" y1="4.5" x2="99" y2="14" width="0.1524" layer="16"/>
+<wire x1="92" y1="4.5" x2="99" y2="4.5" width="0.1524" layer="16"/>
+<wire x1="89" y1="1.5" x2="92" y2="4.5" width="0.1524" layer="16"/>
+<wire x1="37" y1="1.5" x2="89" y2="1.5" width="0.1524" layer="16"/>
+<wire x1="36" y1="2.5" x2="37" y2="1.5" width="0.1524" layer="16"/>
+<wire x1="80.5" y1="10.5" x2="80.43" y2="10.16" width="0.1524" layer="1"/>
+<wire x1="36" y1="2.5" x2="35.56" y2="2.54" width="0.1524" layer="16"/>
+<wire x1="32" y1="2.5" x2="31.52" y2="2.54" width="0.1524" layer="1"/>
+<via x="80.5" y="11.5" extent="1-16" drill="0.2"/>
 </signal>
 <signal name="LED2">
 <contactref element="R2" pad="1"/>
-<wire x1="73.75" y1="11.75" x2="75.25" y2="10.25" width="0.1524" layer="1"/>
+<wire x1="73.75" y1="11.75" x2="74.5" y2="11" width="0.1524" layer="1"/>
+<wire x1="74.5" y1="11" x2="75.25" y2="10.25" width="0.1524" layer="1"/>
 <wire x1="73.75" y1="27.25" x2="73.75" y2="11.75" width="0.1524" layer="1"/>
-<wire x1="72.75" y1="28.25" x2="73.75" y2="27.25" width="0.1524" layer="16"/>
-<wire x1="37" y1="28.25" x2="72.75" y2="28.25" width="0.1524" layer="16"/>
-<wire x1="35.75" y1="29.5" x2="37" y2="28.25" width="0.1524" layer="16"/>
-<wire x1="12.5" y1="29.5" x2="35.75" y2="29.5" width="0.1524" layer="16"/>
-<wire x1="6.5" y1="35.5" x2="12.5" y2="29.5" width="0.1524" layer="16"/>
 <wire x1="75.25" y1="10.25" x2="75.35" y2="10.16" width="0.1524" layer="1"/>
 <via x="73.75" y="27.25" extent="1-16" drill="0.2"/>
 <contactref element="U$2" pad="GPIO7"/>
 <contactref element="PIN_R" pad="18"/>
-<wire x1="31.75" y1="5" x2="35.5" y2="5" width="0.1524" layer="1"/>
+<wire x1="32" y1="5" x2="35.5" y2="5" width="0.1524" layer="1"/>
 <wire x1="35.5" y1="5" x2="35.56" y2="5.08" width="0.1524" layer="1"/>
-<wire x1="31.52" y1="5.08" x2="6.5" y2="35.5" width="0" layer="19" extent="16-16"/>
-<wire x1="31.75" y1="5" x2="31.52" y2="5.08" width="0" layer="19" extent="1-1"/>
+<wire x1="32" y1="5" x2="31.52" y2="5.08" width="0.1524" layer="1"/>
+<wire x1="37" y1="5" x2="36" y2="5" width="0.1524" layer="1"/>
+<wire x1="37" y1="2.5" x2="37" y2="5" width="0.1524" layer="1"/>
+<wire x1="37.5" y1="3" x2="37" y2="2.5" width="0.1524" layer="16"/>
+<wire x1="90" y1="3" x2="37.5" y2="3" width="0.1524" layer="16"/>
+<wire x1="91.5" y1="4.5" x2="90" y2="3" width="0.1524" layer="16"/>
+<wire x1="91.5" y1="6.5" x2="91.5" y2="4.5" width="0.1524" layer="16"/>
+<wire x1="89.5" y1="6.5" x2="91.5" y2="6.5" width="0.1524" layer="16"/>
+<wire x1="89" y1="6" x2="89.5" y2="6.5" width="0.1524" layer="16"/>
+<wire x1="89" y1="4.5" x2="89" y2="6" width="0.1524" layer="16"/>
+<wire x1="88.5" y1="4" x2="89" y2="4.5" width="0.1524" layer="16"/>
+<wire x1="82.5" y1="4" x2="88.5" y2="4" width="0.1524" layer="16"/>
+<wire x1="75" y1="11.5" x2="82.5" y2="4" width="0.1524" layer="16"/>
+<wire x1="74.5" y1="11" x2="75" y2="11.5" width="0.1524" layer="1"/>
+<wire x1="36" y1="5" x2="35.56" y2="5.08" width="0.1524" layer="1"/>
+<via x="37" y="2.5" extent="1-16" drill="0.2"/>
+<via x="75" y="11.5" extent="1-16" drill="0.2"/>
 </signal>
 <signal name="SERVO1">
@@
 <wire x1="35.5" y1="12.75" x2="35.56" y2="12.7" width="0.1524" layer="1"/>
 <wire x1="31.75" y1="12.75" x2="31.52" y2="12.7" width="0.1524" layer="1"/>
-<wire x1="35.75" y1="12.75" x2="35.56" y2="12.7" width="0.1524" layer="1"/>
 <wire x1="78.5" y1="33" x2="78.5" y2="32.5" width="0.1524" layer="1"/>
 <wire x1="73.5" y1="38" x2="78.5" y2="33" width="0.1524" layer="1"/>
@@
 <wire x1="31.75" y1="10.25" x2="31.52" y2="10.16" width="0.1524" layer="1"/>
 <wire x1="35.5" y1="10.25" x2="35.56" y2="10.16" width="0.1524" layer="1"/>
-<wire x1="35.75" y1="10.25" x2="35.56" y2="10.16" width="0.1524" layer="1"/>
 <via x="78" y="20.5" extent="1-16" drill="0.2"/>
 </signal>
@@
 <contactref element="U$9" pad="CSB"/>
 <contactref element="PIN_L" pad="1"/>
-<wire x1="6.25" y1="48.5" x2="2.75" y2="52" width="0.1524" layer="1"/>
-<wire x1="2.75" y1="52" x2="2.54" y2="52.07" width="0.1524" layer="1"/>
 <wire x1="75.5" y1="23.25" x2="75.5" y2="28.25" width="0.1524" layer="1"/>
 <wire x1="77" y1="21.75" x2="75.5" y2="23.25" width="0.1524" layer="16"/>
@@
 <wire x1="98" y1="11.5" x2="97.79" y2="11.43" width="0.1524" layer="1"/>
 <wire x1="98" y1="21.5" x2="97.79" y2="21.59" width="0.1524" layer="1"/>
-<wire x1="23.25" y1="31.5" x2="6.5" y2="48.25" width="0.1524" layer="16"/>
-<wire x1="59.25" y1="31.5" x2="23.25" y2="31.5" width="0.1524" layer="16"/>
+<wire x1="59.25" y1="31.5" x2="31" y2="31.5" width="0.1524" layer="16"/>
 <wire x1="60.5" y1="30.25" x2="59.25" y2="31.5" width="0.1524" layer="16"/>
 <wire x1="77.25" y1="30.25" x2="60.5" y2="30.25" width="0.1524" layer="16"/>
@@
 <via x="75.5" y="23.25" extent="1-16" drill="0.2"/>
 <contactref element="RASPBERRYPI_4B" pad="3V3_1"/>
-<wire x1="6.25" y1="48.5" x2="10.16" y2="52.07" width="0" layer="19" extent="1-1"/>
-<wire x1="6.5" y1="48.25" x2="6.25" y2="48.5" width="0" layer="19" extent="1-16"/>
+<wire x1="10" y1="52" x2="3" y2="52" width="0.1524" layer="1"/>
+<wire x1="3" y1="52" x2="2.54" y2="52.07" width="0.1524" layer="1"/>
+<wire x1="10" y1="52" x2="10.16" y2="52.07" width="0.1524" layer="1"/>
+<wire x1="31" y1="31.5" x2="10.5" y2="52" width="0.1524" layer="16"/>
+<wire x1="10.5" y1="52" x2="10.16" y2="52.07" width="0.1524" layer="16"/>
 </signal>
 <signal name="+5V">
@@
 <contactref element="U$2" pad="GPIO34"/>
 <contactref element="PIN_L" pad="5"/>
-<wire x1="6.25" y1="38.25" x2="2.75" y2="41.75" width="0.1524" layer="1"/>
+<wire x1="6" y1="38.5" x2="2.75" y2="41.75" width="0.1524" layer="1"/>
 <wire x1="2.75" y1="41.75" x2="2.54" y2="41.91" width="0.1524" layer="1"/>
-<wire x1="6.25" y1="38.25" x2="6.35" y2="38.1" width="0" layer="19" extent="1-1"/>
+<wire x1="6" y1="38.5" x2="6.35" y2="38.1" width="0.1524" layer="1"/>
 </signal>
 <signal name="IO35">
 <contactref element="U$2" pad="GPIO35"/>
 <contactref element="PIN_L" pad="6"/>
-<wire x1="6.25" y1="35.75" x2="2.75" y2="39.25" width="0.1524" layer="1"/>
+<wire x1="6" y1="36" x2="2.75" y2="39.25" width="0.1524" layer="1"/>
 <wire x1="2.75" y1="39.25" x2="2.54" y2="39.37" width="0.1524" layer="1"/>
-<wire x1="6.25" y1="35.75" x2="6.35" y2="35.56" width="0" layer="19" extent="1-1"/>
+<wire x1="6" y1="36" x2="6.35" y2="35.56" width="0.1524" layer="1"/>
 </signal>
 </signals>
