File: NSE2022/Eagle/PCB/runback_ver2.0/ranback_top.brd (EAGLE design)
At the start: 100 x 61.3 mm, 25 parts

Commit message: ssad
Routing:
- net BB_SDA: track 0.00 -> 126.3 mm
- net +3V3: track 0.00 -> 121.4 mm, vias 0 -> 1
- net BB_SCL: track 0.00 -> 120.1 mm, vias 0 -> 2
- net MD_LB: track 0.00 -> 76.2 mm, vias 0 -> 3
- net N$6: track 0.00 -> 65.1 mm, vias 0 -> 4
- net MD_LF: track 0.00 -> 63.4 mm, vias 0 -> 2
- net SERVO2: track 0.00 -> 62.8 mm
- net SERVO1: track 0.00 -> 60.6 mm
- net IM_BUSY: track 0.00 -> 60.3 mm, vias 0 -> 1
- net LED6: track 0.00 -> 56.2 mm, vias 0 -> 2
- net N$5: track 0.00 -> 54.9 mm, vias 0 -> 3
- net IM_RESET: track 0.00 -> 53.2 mm, vias 0 -> 1
- net LED5: track 0.00 -> 52.5 mm, vias 0 -> 1
- net LED4: track 0.00 -> 49.8 mm, vias 0 -> 1
- net RP_RX: track 0.00 -> 49.2 mm, vias 0 -> 3
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