File: NSE2022/Eagle/PCB/runback_ver2.0/ranback_top.brd (EAGLE design)
At the start: 100 x 61.3 mm, 25 parts

Commit message: asd
Connections:
- removed net IO5: PIN_R.10, U$2.GPIO5
- new net IO39: PIN_L.4, U$2.GPIO39
- net RP_SS: now also PIN_R.10, U$2.GPIO5; no longer PIN_L.4, U$2.GPIO39
Routing:
- net IO39: track 0.00 -> 30.2 mm
- net RP_SS: track 45.6 -> 57.6 mm, vias 0 -> 2
- net IO5: track 7.43 -> 0.00 mm
Changed lines of the file:
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@@
 <signal name="RP_SS">
 <contactref element="RASPBERRYPI_4B" pad="GPIO8"/>
-<contactref element="U$2" pad="GPIO39"/>
-<contactref element="PIN_L" pad="4"/>
-<wire x1="63.75" y1="41.75" x2="64.75" y2="40.75" width="0.1524" layer="1"/>
-<wire x1="37.5" y1="41.75" x2="63.75" y2="41.75" width="0.1524" layer="1"/>
-<wire x1="36.5" y1="40.75" x2="37.5" y2="41.75" width="0.1524" layer="1"/>
-<wire x1="35.75" y1="40.75" x2="36.5" y2="40.75" width="0.1524" layer="1"/>
-<wire x1="64.75" y1="40.75" x2="64.77" y2="40.64" width="0.1524" layer="1"/>
-<wire x1="35.75" y1="40.75" x2="35.56" y2="40.64" width="0.1524" layer="1"/>
-<wire x1="36.5" y1="53" x2="38" y2="54.5" width="0.1524" layer="16"/>
-<wire x1="36.5" y1="51" x2="36.5" y2="53" width="0.1524" layer="16"/>
-<wire x1="37" y1="50.5" x2="36.5" y2="51" width="0.1524" layer="16"/>
-<wire x1="37" y1="42.25" x2="37" y2="50.5" width="0.1524" layer="16"/>
-<wire x1="35.75" y1="41" x2="37" y2="42.25" width="0.1524" layer="16"/>
-<wire x1="35.75" y1="40.75" x2="35.75" y2="41" width="0.1524" layer="16"/>
-<wire x1="38" y1="54.5" x2="38.1" y2="54.61" width="0.1524" layer="16"/>
-<wire x1="35.75" y1="40.75" x2="35.56" y2="40.64" width="0.1524" layer="16"/>
+<contactref element="U$2" pad="GPIO5"/>
+<contactref element="PIN_R" pad="10"/>
+<wire x1="38.1" y1="54.61" x2="39.37" y2="53.34" width="0.1524" layer="1"/>
+<wire x1="39.37" y1="53.34" x2="39.37" y2="48.81105625" width="0.1524" layer="1"/>
+<wire x1="39.37" y1="48.81105625" x2="39.92105625" y2="48.26" width="0.1524" layer="1"/>
+<wire x1="39.92105625" y1="48.26" x2="48.26" y2="48.26" width="0.1524" layer="1"/>
+<via x="48.26" y="48.26" extent="1-16" drill="0.35"/>
+<wire x1="48.26" y1="48.26" x2="51.4452" y2="45.0748" width="0.1524" layer="16"/>
+<wire x1="51.4452" y1="45.0748" x2="51.4452" y2="28.12374375" width="0.1524" layer="16"/>
+<wire x1="52.07" y1="27.49894375" x2="52.07" y2="24.13" width="0.1524" layer="16"/>
+<wire x1="51.4452" y1="28.12374375" x2="52.07" y2="27.49894375" width="0.1524" layer="16"/>
+<via x="52.07" y="24.13" extent="1-16" drill="0.35"/>
+<wire x1="52.07" y1="24.13" x2="52.8852" y2="24.9452" width="0.1524" layer="1"/>
+<wire x1="52.8852" y1="24.9452" x2="54.12625625" y2="24.9452" width="0.1524" layer="1"/>
+<wire x1="54.58105625" y1="25.4" x2="60.73" y2="25.4" width="0.1524" layer="1"/>
+<wire x1="54.12625625" y1="24.9452" x2="54.58105625" y2="25.4" width="0.1524" layer="1"/>
+<wire x1="64.0213125" y1="24.5174" x2="65.5186875" y2="24.5174" width="0.1524" layer="1"/>
+<wire x1="60.73" y1="25.4" x2="63.1387125" y2="25.4" width="0.1524" layer="1"/>
+<wire x1="66.4012875" y1="25.4" x2="67.31" y2="25.4" width="0.1524" layer="1"/>
+<wire x1="63.1387125" y1="25.4" x2="64.0213125" y2="24.5174" width="0.1524" layer="1"/>
+<wire x1="65.5186875" y1="24.5174" x2="66.4012875" y2="25.4" width="0.1524" layer="1"/>
 </signal>
 <signal name="LED1">
@@
 <wire x1="35.75" y1="12.75" x2="35.56" y2="12.7" width="0.1524" layer="1"/>
 </signal>
-<signal name="IO5">
-<contactref element="U$2" pad="GPIO5"/>
-<contactref element="PIN_R" pad="10"/>
-<wire x1="66.5" y1="24.5" x2="67.25" y2="25.25" width="0.1524" layer="1"/>
-<wire x1="64" y1="24.5" x2="66.5" y2="24.5" width="0.1524" layer="1"/>
-<wire x1="63.25" y1="25.25" x2="64" y2="24.5" width="0.1524" layer="1"/>
-<wire x1="60.75" y1="25.25" x2="63.25" y2="25.25" width="0.1524" layer="1"/>
-<wire x1="67.25" y1="25.25" x2="67.31" y2="25.4" width="0.1524" layer="1"/>
-<wire x1="60.75" y1="25.25" x2="60.73" y2="25.4" width="0.1524" layer="1"/>
-</signal>
 <signal name="BB_SDA">
 <contactref element="RASPBERRYPI_4B" pad="GPIO2"/>
@@
 <via x="62.75" y="11.5" extent="1-16" drill="0.35"/>
 </signal>
+<signal name="IO39">
+<contactref element="U$2" pad="GPIO39"/>
+<contactref element="PIN_L" pad="4"/>
+<wire x1="64.75" y1="40.75" x2="63.75" y2="41.75" width="0.1524" layer="1"/>
+<wire x1="64.75" y1="40.75" x2="64.77" y2="40.64" width="0.1524" layer="1"/>
+<wire x1="36.67" y1="41.75" x2="35.56" y2="40.64" width="0.1524" layer="1"/>
+<wire x1="63.75" y1="41.75" x2="36.67" y2="41.75" width="0.1524" layer="1"/>
+</signal>
 </signals>
