File: NSE2022/Eagle/PCB/Rocket_ver2/NSE2022_GPSDOWNLINK_ver0.brd (EAGLE design)
At the start: 85 x 85 mm, 31 parts, among them CN2 DM3AT

Commit message: aaa
Parts:
- removed SRIDE_SWTCH3: SRIDE_SWITCH, Switches:SRIDE_SWITCH
- added U$8: SLIDESWITCH, SLIDESWITCH:SLIDESWITCH
Connections:
- net N$12: now also U$8.A; no longer SRIDE_SWTCH3.L
- net N$4: now also U$8.C; no longer SRIDE_SWTCH3.LR
Routing:
- net GND: track 241.6 -> 33.9 mm, vias 0 -> 4
- net +5V: track 161.6 -> 111.8 mm
- net IMTX: track 79.2 -> 59.9 mm, vias 0 -> 2
- net FP: track 90.2 -> 72.2 mm
- net N$9: track 73.2 -> 55.9 mm, vias 1 -> 2
- net +3V3: track 96.5 -> 80.7 mm
- net SCK: track 62.7 -> 47.8 mm, vias 0 -> 2
- net N$4: track 99.8 -> 86.3 mm, vias 0 -> 1
- net CANL2: track 37.6 -> 24.9 mm
- net CANL2OUT: track 66.2 -> 56.9 mm, vias 0 -> 2
- net SS: track 60.6 -> 51.7 mm, vias 0 -> 2
- net SDA: track 61.4 -> 69.0 mm
- net MISO: track 47.1 -> 40.1 mm, vias 0 -> 1
- net CANH2OUT: track 70.9 -> 64.2 mm, vias 0 -> 2
- net GPSRX: track 88.3 -> 93.0 mm
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- added copper zone on layer 1, net GND
- added copper zone on layer 16, net GND
