File: NSE2022/Eagle/PCB/Rocket_ver2/NSE2022_BATTERY_ver0.brd (EAGLE design)
At the start: 85 x 85 mm, 16 parts

Commit message: a
Routing:
- net BPIN3: track 95.0 -> 161.5 mm, vias 1 -> 0
- net APIN1: track 79.5 -> 110.1 mm, vias 3 -> 0
- net APIN3: track 96.9 -> 122.3 mm, vias 1 -> 0
- net APIN2: track 98.3 -> 77.3 mm, vias 1 -> 2
- net 6V-OUT: track 93.4 -> 113.5 mm
- net N$13: track 48.0 -> 65.5 mm, vias 1 -> 0
- net 3V+IN: track 93.9 -> 78.1 mm
- net 6V+OUT: track 87.4 -> 102.0 mm, vias 0 -> 1
- net BPIN1: track 82.4 -> 90.9 mm, vias 2 -> 1
- net FP+IN: track 91.4 -> 96.2 mm
- net BPIN2: track 82.2 -> 80.3 mm
- net 6V+IN: track 89.0 -> 87.4 mm
- net 3V+OUT: track 77.5 -> 78.5 mm
- net FP-IN: track 87.5 -> 86.5 mm
- removed copper zone on layer 1, net GND
- removed copper zone on layer 16, net GND
