File: NSE2022/Eagle/PCB/Rocket_ver2/NSE2022_ROCKETCONTROLLER_ver0.brd (EAGLE design)
At the start: 85 x 85 mm, 41 parts, among them CN1 DM3AT

Commit message: rc_brd_kato
Parts:
- removed SRIDE_SWTCH1, SRIDE_SWTCH2: SRIDE_SWITCH, Switches:SRIDE_SWITCH
- added U$2, U$3: SLIDESWITCH, SLIDESWITCH:SLIDESWITCH
- moved U$30 57.9 mm to (28.7, 8.00), turned to 270 degrees
- moved U$13 57.7 mm to (-20.5, -23.3), turned to 0 degrees
- moved U$21 29.0 mm to (-17.5, 32.9)
- moved U$20 28.5 mm to (11.1, 33.4)
- moved U$12 3.35 mm to (-20.5, -18.1)
- moved CERAMIC_CAPACITOR6 1.58 mm to (-33.3, 14.5)
- moved CERAMIC_CAPACITOR4 1.12 mm to (-22.2, 14.5)
- moved CERAMIC_CAPACITOR5 1.12 mm to (-27.6, 14.5)
- moved CERAMIC_CAPACITOR3 0.50 mm to (-16.7, 14.5)
Connections:
- net N$10: now also U$2.A; no longer SRIDE_SWTCH2.L
- net N$11: now also U$3.A; no longer SRIDE_SWTCH1.L
- net N$24: now also U$2.C; no longer SRIDE_SWTCH2.LR
- net N$6: now also U$3.C; no longer SRIDE_SWTCH1.LR
Routing:
- net GND: track 322.9 -> 19.8 mm, vias 0 -> 2
- net N$22: track 111.4 -> 9.92 mm
- net N$2: track 91.0 -> 5.26 mm
- net SCK: track 42.8 -> 85.5 mm, vias 0 -> 1
- net SERVO5V: track 140.4 -> 105.1 mm, vias 1 -> 0
- net +3V3: track 168.9 -> 140.4 mm, vias 0 -> 1
- net BATTE_SERVO: track 32.7 -> 60.9 mm
- net BATTE_RC: track 61.0 -> 36.1 mm
- net N$6: track 44.9 -> 62.6 mm, vias 0 -> 1
- net +5V: track 136.9 -> 119.3 mm, vias 0 -> 1
- net N$11: track 46.0 -> 62.5 mm
- net MISO: track 41.3 -> 56.4 mm, vias 0 -> 3
- net MOSI: track 69.2 -> 56.7 mm
- net CANL1: track 44.5 -> 56.9 mm
- net SERVO1: track 57.9 -> 70.0 mm, vias 0 -> 1
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- added copper zone on layer 1, net GND
- added copper zone on layer 16, net GND
Other:
- board text added: "RC"
- board text added: "servo"

Commit message: a
Routing:
- net N$15: track 48.6 -> 49.9 mm
- net +3V3: track 140.4 -> 141.3 mm
- net SERVO3: track 49.8 -> 50.6 mm
- net SERVO1: track 70.0 -> 70.7 mm
- net SS: track 57.2 -> 57.8 mm
