File: NSE2023/EAGLE/project/STM32F3_Motherver/Rocket Controller ver1.0.1.sch (EAGLE design)
At the start: 23 parts

Commit message: a
Connections:
- new net FP_CHECKER: JP3.15, U$1.PB4
- net PWM: no longer JP3.15
Changed lines of the file:
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@@
-</segment>
-<segment>
-<pinref part="JP3" gate="A" pin="15"/>
-<wire x1="106.68" y1="-22.86" x2="101.6" y2="-22.86" width="0.1524" layer="91"/>
-<label x="101.6" y="-22.86" size="1.778" layer="95" rot="R180" xref="yes"/>
 </segment>
 <segment>
@@
 </segment>
 </net>
+<net name="FP_CHECKER" class="0">
+<segment>
+<pinref part="JP3" gate="A" pin="15"/>
+<wire x1="106.68" y1="-22.86" x2="101.6" y2="-22.86" width="0.1524" layer="91"/>
+<label x="101.6" y="-22.86" size="1.778" layer="95" rot="R180" xref="yes"/>
+</segment>
+<segment>
+<pinref part="U$1" gate="G$1" pin="PB4"/>
+<wire x1="60.96" y1="60.96" x2="76.2" y2="60.96" width="0.1524" layer="91"/>
+<label x="76.2" y="60.96" size="1.778" layer="95" xref="yes"/>
+</segment>
+</net>
