File: NSE2023/EAGLE/project/STM32F3_Motherver/Down Linker ver1.0.0.sch (EAGLE design)
At the start: 27 parts

Commit message: a
Connections:
- new net FP_CHECKER: JP3.15, U$1.PB4
- net PWM: no longer JP3.15
- net SCL: now also U$1.PA15/I2C1_SCL
- net SDA: now also U$1.PB7/I2C1_SDA
Changed lines of the file:
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@@
 <attribute name="VALUE" x="162.56" y="15.24" size="1.778" layer="96" rot="R90"/>
 </instance>
-<instance part="P+2" gate="1" x="83.82" y="-20.32" smashed="yes">
-<attribute name="VALUE" x="81.28" y="-25.4" size="1.778" layer="96" rot="R90"/>
+<instance part="P+2" gate="1" x="78.74" y="-20.32" smashed="yes">
+<attribute name="VALUE" x="76.2" y="-25.4" size="1.778" layer="96" rot="R90"/>
 </instance>
 <instance part="P+3" gate="1" x="119.38" y="2.54" smashed="yes">
@@
 <pinref part="JP3" gate="A" pin="18"/>
 </segment>
+<segment>
+<pinref part="U$1" gate="G$1" pin="PB7/I2C1_SDA"/>
+<wire x1="60.96" y1="76.2" x2="73.66" y2="76.2" width="0.1524" layer="91"/>
+<label x="73.66" y="76.2" size="1.778" layer="95" xref="yes"/>
+</segment>
 </net>
 <net name="NRST" class="0">
@@
 <pinref part="JP3" gate="A" pin="16"/>
 </segment>
+<segment>
+<pinref part="U$1" gate="G$1" pin="PA15/I2C1_SCL"/>
+<wire x1="60.96" y1="50.8" x2="76.2" y2="50.8" width="0.1524" layer="91"/>
+<label x="76.2" y="50.8" size="1.778" layer="95" xref="yes"/>
+</segment>
 </net>
 <net name="SWCLK" class="0">
@@
 </net>
 <net name="PWM" class="0">
-<segment>
-<pinref part="JP3" gate="A" pin="15"/>
-<wire x1="106.68" y1="-22.86" x2="101.6" y2="-22.86" width="0.1524" layer="91"/>
-<label x="101.6" y="-22.86" size="1.778" layer="95" rot="R180" xref="yes"/>
-</segment>
 <segment>
 <wire x1="114.3" y1="-10.16" x2="119.38" y2="-10.16" width="0.1524" layer="91"/>
@@
 <pinref part="P+2" gate="1" pin="+5V"/>
 <pinref part="JP3" gate="A" pin="17"/>
-<wire x1="83.82" y1="-22.86" x2="83.82" y2="-25.4" width="0.1524" layer="91"/>
-<wire x1="83.82" y1="-25.4" x2="106.68" y2="-25.4" width="0.1524" layer="91"/>
+<wire x1="78.74" y1="-22.86" x2="78.74" y2="-25.4" width="0.1524" layer="91"/>
+<wire x1="78.74" y1="-25.4" x2="106.68" y2="-25.4" width="0.1524" layer="91"/>
 </segment>
 <segment>
@@
 </segment>
 </net>
+<net name="FP_CHECKER" class="0">
+<segment>
+<pinref part="JP3" gate="A" pin="15"/>
+<wire x1="106.68" y1="-22.86" x2="101.6" y2="-22.86" width="0.1524" layer="91"/>
+<label x="101.6" y="-22.86" size="1.778" layer="95" rot="R180" xref="yes"/>
+</segment>
+<segment>
+<pinref part="U$1" gate="G$1" pin="PB4"/>
+<wire x1="60.96" y1="60.96" x2="76.2" y2="60.96" width="0.1524" layer="91"/>
+<label x="76.2" y="60.96" size="1.778" layer="95" xref="yes"/>
+</segment>
+</net>
