File: NSE2023/EAGLE/project/STM32F3_Motherver/Mother Board.brd (EAGLE design)
At the start: 54.5 x 54.5 mm, 32 parts

Commit message: death
Parts:
- added CON8: (no value), XR Connector:3PIN
- added POLYSWITCH1: (no value), pinhead:1X02
- moved R2 93.1 mm to (8.50, 13.0), turned to 180 degrees
- moved C2 84.0 mm to (3.00, 24.0)
- moved POLYSWITCH 83.5 mm to (24.0, -0.18), turned to 90 degrees
- moved C1 81.4 mm to (-5.50, 24.0)
- moved R1 80.4 mm to (-6.00, 13.0), turned to 180 degrees
- moved R4 76.7 mm to (-15.5, 4.00), turned to 180 degrees
- moved MOS5 75.9 mm to (-3.74, -17.9)
- moved R5 74.3 mm to (-15.5, -4.00), turned to 180 degrees
- moved R6 74.2 mm to (-7.00, -16.5)
- moved CON2 68.1 mm to (18.1, -4.07), flipped to the bottom, turned to 270 degrees
- moved R3 63.2 mm to (-7.00, -19.0), turned to 180 degrees
- moved MOS2 62.6 mm to (-15.9, -0.30), turned to 180 degrees
- moved CON1 60.9 mm to (18.1, -12.0), flipped to the bottom, turned to 270 degrees
- moved U$2 56.9 mm to (-2.13, -22.9), turned to 180 degrees
- moved C3 55.9 mm to (-9.50, -17.5), turned to 90 degrees
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Connections:
- new net 5V_RAW: CON8.P$2, POLYSWITCH1.2
- net +3V3: now also PS1.P$19, PS1.P$2, PS2.P$19, PS2.P$2, PS3.P$19, PS3.P$2; no longer PS1.P$1, PS1.P$20, PS2.P$1, PS2.P$20, PS3.P$1, PS3.P$20
- net +5V: now also POLYSWITCH1.1, PS1.P$18, PS1.P$3, PS2.P$18, PS2.P$3, PS3.P$18, PS3.P$3; no longer PS1.P$17, PS1.P$4, PS2.P$17, PS2.P$4, PS3.P$17, PS3.P$4
- net BIT1: now also PS1.P$12, PS1.P$9, PS2.P$12, PS2.P$9, PS3.P$12, PS3.P$9; no longer PS1.P$10, PS1.P$11, PS2.P$10, PS2.P$11, PS3.P$10, PS3.P$11
- net BIT2: now also PS1.P$14, PS1.P$7, PS2.P$14, PS2.P$7, PS3.P$14, PS3.P$7; no longer PS1.P$13, PS1.P$8, PS2.P$13, PS2.P$8, PS3.P$13, PS3.P$8
- net FP_CHECKER: now also PS1.P$5, PS2.P$5, PS3.P$5; no longer PS1.P$15, PS2.P$15, PS3.P$15
- net GND: now also CON8.P$1, PS1.P$1, PS1.P$20, PS2.P$1, PS2.P$20, PS3.P$1, PS3.P$20; no longer PS1.P$19, PS1.P$2, PS2.P$19, PS2.P$2, PS3.P$19, PS3.P$2
- net LOGRX: now also PS1.P$13, PS1.P$8, PS2.P$13, PS2.P$8, PS3.P$13, PS3.P$8; no longer PS1.P$14, PS1.P$7, PS2.P$14, PS2.P$7, PS3.P$14, PS3.P$7
- net LOGTX: now also PS1.P$10, PS1.P$11, PS2.P$10, PS2.P$11, PS3.P$10, PS3.P$11; no longer PS1.P$12, PS1.P$9, PS2.P$12, PS2.P$9, PS3.P$12, PS3.P$9
- net PWM: now also CON8.P$3, PS1.P$16, PS2.P$16, PS3.P$16; no longer PS1.P$6, PS2.P$6, PS3.P$6
- net SCL0: now also PS1.P$15, PS1.P$6; no longer PS3.P$16, PS3.P$5
- net SCL1: now also PS2.P$15, PS2.P$6; no longer PS2.P$16, PS2.P$5
- net SCL2: now also PS3.P$15, PS3.P$6; no longer PS1.P$16, PS1.P$5
- net SDA0: now also PS1.P$17, PS1.P$4; no longer PS3.P$18, PS3.P$3
- net SDA1: now also PS2.P$17, PS2.P$4; no longer PS2.P$18, PS2.P$3
- net SDA2: now also PS3.P$17, PS3.P$4; no longer PS1.P$18, PS1.P$3
Routing:
- net GND: track 0.00 -> 179.8 mm
- net FP: track 0.00 -> 155.9 mm, vias 0 -> 1
- net +3V3: track 0.00 -> 141.9 mm
- net +5V: track 0.00 -> 90.6 mm, vias 0 -> 1
- net BIT2: track 0.00 -> 59.5 mm
- net LOGRX: track 0.00 -> 55.6 mm
- net 7.4_1ENT: track 0.00 -> 49.8 mm
- net 7.4_0ENT: track 0.00 -> 47.2 mm
- net BIT1: track 0.00 -> 46.8 mm
- net 5V_ENT: track 0.00 -> 45.7 mm
- net FP_CHECKER: track 0.00 -> 33.8 mm
- net SDA2: track 0.00 -> 32.7 mm
- net SDA1: track 0.00 -> 32.6 mm
- net PWM: track 0.00 -> 31.9 mm
- net SDA0: track 0.00 -> 30.7 mm
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- added copper zone on layer 1, net GND
- added copper zone on layer 16, net GND
Other:
- board size 54.5 x 54.5 mm -> 54 x 54 mm
