File: NSE2023/EAGLE/project/STM32F3_Motherver/Mother Board.sch (EAGLE design)
At the start: 3 parts

Commit message: a
Parts:
- added C1, C2: 3.3uF, rcl:C-USC0603
- added C3: 10uF, rcl:C-USC0603
- added CON1, CON2, CON3, CON4, CON5, CON6, CON7: (no value), XR Connector:2PIN
- added D1, D2: 1N4148DO35-7, diode:1N4148DO35-7
- added DCDC1: (no value), DC-DC:5V1A_M78AR05-1
- added DCDC2: (no value), DC-DC:3.3V1A_M78AR033-1
- added MOS1, MOS2, MOS3, MOS4, MOS5, MOS6, MOS7: (no value), Chip MOSFET:PCH_SSM6J808R
- added POLYSWITCH: (no value), pinhead:PINHD-1X2
- added R1, R2, R3: 1k, rcl:R-US_R0603
- added R4, R5: 100k, rcl:R-US_R0603
- added R6: 10k, rcl:R-US_R0603
- added U$2: 1X4, PinSocket:1X4
Connections:
- new net +3V3: MOS2.1, MOS2.2, MOS2.5, MOS2.6, MOS5.4, POLYSWITCH.1, PS1.P$1, PS1.P$20, PS2.P$1, PS2.P$20, PS3.P$1, PS3.P$20
- new net +5V: MOS1.1, MOS1.2, MOS1.5, MOS1.6, PS1.P$17, PS1.P$4, PS2.P$17, PS2.P$4, PS3.P$17, PS3.P$4
- new net 3.3VSW: CON7.P$2, MOS2.3, R5.1
- new net 3.3V_ENT: C2.1, DCDC2.VOUT
- new net 3.3_RAW: CON4.P$2, POLYSWITCH.2
- new net 5VSW: CON6.P$2, MOS1.3, R4.1
- new net 5V_ENT: C1.1, DCDC1.VOUT, MOS1.4, R4.2
- new net 5V_ENT1: MOS2.4, R5.2
- new net 7.4_0ENT: MOS7.4, U$2.P$3
- new net 7.4_1ENT: MOS4.4, U$2.P$5
- new net BIT1: PS1.P$10, PS1.P$11, PS2.P$10, PS2.P$11, PS3.P$10, PS3.P$11
- new net BIT2: PS1.P$13, PS1.P$8, PS2.P$13, PS2.P$8, PS3.P$13, PS3.P$8
- new net FP: CON5.P$2, D1.A, D2.A, MOS3.3, MOS4.3, MOS5.3, MOS6.3, MOS7.3, R1.2, R2.2, U$2.P$1
- new net FP_CHECKER: C3.1, PS1.P$15, PS2.P$15, PS3.P$15, R3.2
- new net GND: C1.2, C2.2, C3.2, CON4.P$1, CON5.P$1, CON6.P$1, CON7.P$1, DCDC1.GND, DCDC2.GND, PS1.P$19, PS1.P$2, PS2.P$19, PS2.P$2, PS3.P$19, PS3.P$2, R1.1, R2.1, R6.1, U$2.P$7
- new net LOGRX: PS1.P$14, PS1.P$7, PS2.P$14, PS2.P$7, PS3.P$14, PS3.P$7
- new net LOGTX: PS1.P$12, PS1.P$9, PS2.P$12, PS2.P$9, PS3.P$12, PS3.P$9
- new net N$1: D2.C, DCDC2.VIN, MOS6.4
- new net N$11: D1.C, DCDC1.VIN, MOS3.4
- new net N$12: MOS3.1, MOS3.2, MOS3.5, MOS3.6, MOS7.1, MOS7.2, MOS7.5, MOS7.6
- new net N$14: MOS5.1, MOS5.2, MOS5.5, MOS5.6, R3.1, R6.2
- new net N$2: MOS4.1, MOS4.2, MOS4.5, MOS4.6, MOS6.1, MOS6.2, MOS6.5, MOS6.6
- new net PWM: PS1.P$6, PS2.P$6, PS3.P$6
- new net SCL0: CON1.P$1, PS3.P$16, PS3.P$5
- new net SCL1: CON2.P$1, PS2.P$16, PS2.P$5
- new net SCL2: CON3.P$1, PS1.P$16, PS1.P$5
- new net SDA0: CON1.P$2, PS3.P$18, PS3.P$3
- new net SDA1: CON2.P$2, PS2.P$18, PS2.P$3
- new net SDA2: CON3.P$2, PS1.P$18, PS1.P$3
Other:
- moved on the sheet: PS1, PS2, PS3

Commit message: death
Parts:
- added CON8: (no value), XR Connector:3PIN
- added POLYSWITCH1: (no value), pinhead:PINHD-1X2
Connections:
- new net 5V_RAW: CON8.P$2, POLYSWITCH1.2
- net +3V3: now also PS1.P$19, PS1.P$2, PS2.P$19, PS2.P$2, PS3.P$19, PS3.P$2; no longer PS1.P$1, PS1.P$20, PS2.P$1, PS2.P$20, PS3.P$1, PS3.P$20
- net +5V: now also POLYSWITCH1.1, PS1.P$18, PS1.P$3, PS2.P$18, PS2.P$3, PS3.P$18, PS3.P$3; no longer PS1.P$17, PS1.P$4, PS2.P$17, PS2.P$4, PS3.P$17, PS3.P$4
- net BIT1: now also PS1.P$12, PS1.P$9, PS2.P$12, PS2.P$9, PS3.P$12, PS3.P$9; no longer PS1.P$10, PS1.P$11, PS2.P$10, PS2.P$11, PS3.P$10, PS3.P$11
- net BIT2: now also PS1.P$14, PS1.P$7, PS2.P$14, PS2.P$7, PS3.P$14, PS3.P$7; no longer PS1.P$13, PS1.P$8, PS2.P$13, PS2.P$8, PS3.P$13, PS3.P$8
- net FP_CHECKER: now also PS1.P$5, PS2.P$5, PS3.P$5; no longer PS1.P$15, PS2.P$15, PS3.P$15
- net GND: now also CON8.P$1, PS1.P$1, PS1.P$20, PS2.P$1, PS2.P$20, PS3.P$1, PS3.P$20; no longer PS1.P$19, PS1.P$2, PS2.P$19, PS2.P$2, PS3.P$19, PS3.P$2
- net LOGRX: now also PS1.P$13, PS1.P$8, PS2.P$13, PS2.P$8, PS3.P$13, PS3.P$8; no longer PS1.P$14, PS1.P$7, PS2.P$14, PS2.P$7, PS3.P$14, PS3.P$7
- net LOGTX: now also PS1.P$10, PS1.P$11, PS2.P$10, PS2.P$11, PS3.P$10, PS3.P$11; no longer PS1.P$12, PS1.P$9, PS2.P$12, PS2.P$9, PS3.P$12, PS3.P$9
- net PWM: now also CON8.P$3, PS1.P$16, PS2.P$16, PS3.P$16; no longer PS1.P$6, PS2.P$6, PS3.P$6
- net SCL0: now also PS1.P$15, PS1.P$6; no longer PS3.P$16, PS3.P$5
- net SCL1: now also PS2.P$15, PS2.P$6; no longer PS2.P$16, PS2.P$5
- net SCL2: now also PS3.P$15, PS3.P$6; no longer PS1.P$16, PS1.P$5
- net SDA0: now also PS1.P$17, PS1.P$4; no longer PS3.P$18, PS3.P$3
- net SDA1: now also PS2.P$17, PS2.P$4; no longer PS2.P$18, PS2.P$3
- net SDA2: now also PS3.P$17, PS3.P$4; no longer PS1.P$18, PS1.P$3
Other:
- moved on the sheet: PS1, PS2, PS3
