File: NSE2023/EAGLE/project/STM32F3_Motherver/water ver2.0.0.sch (EAGLE design)
At the start: 15 parts

Commit message: edit mother board
Parts:
- removed BMP3: BMP180, BMP180:BMP180
- removed CON10: (no value), XR Connector:2PIN
- removed CON8: (no value), XR Connector:3PIN
- removed SRIDE_SWTCH1: SRIDE_SWITCH, Sride Switch:SRIDE_SWITCH
- CON3, CON5: device XR Connector:2PIN -> XR Connector:3PIN
Connections:
- removed net N$1: CON5.P$2, SRIDE_SWTCH1.L
- removed net N$2: CON5.P$1, SRIDE_SWTCH1.LR
- removed net SCL2: BMP3.SCL, CON3.P$2
- removed net SDA2: BMP3.SDA, CON3.P$1
- net +3V3: no longer BMP3.VIN
- net +5V: no longer CON8.P$2
- net FP: no longer CON10.P$1
- net GND: no longer BMP3.GND, CON10.P$2, CON8.P$1
- net PWM: no longer CON8.P$3
