File: NSE2023/EAGLE/project/CANSAT12th/main 1.0.0.sch (EAGLE design)
At the start: 25 parts, among them CN1 DM3AT

Commit message: add
Parts:
- removed IM: IM920C, IM920:IM920C
- removed LED1: (no value), Chip LED:OSXX1608C1A
- removed R4: 100, rcl:R-US_R0603
- removed U$2: AE-GYSFDMAXB, AE-GYSFDMAXB:AE-GYSFDMAXB
- added CON1, CON3: (no value), XR Connector:4PIN_SIDE
- added CON2: (no value), XR Connector:6PIN_SIDE
Connections:
- removed net CAM_SCL: U$1.GP27
- removed net CAM_SDA: CAM.2, U$1.GP26
- removed net GND1: U$2.GND
- removed net LED: IM.STATUS, LED1.AN
- removed net N$1: CAM.8
- removed net N$3: LED1.CT, R4.2
- new net 1: CN1.CLK, R10.2, R6.2
- new net ECHO: CON3.P$3, U$1.GP26
- new net TRIG: CON3.P$1, U$1.GP27
- net +12V: no longer PIXY2.P$3
- net +3V3: now also CON2.P$6; no longer IM.VCC
- net +5V: now also CON1.P$2, CON3.P$2, PIXY2.P$3; no longer U$2.5V
- net CAM_NSS: now also CAM.8
- net CAM_SCK: no longer CAM.1
- net GND: now also CON1.P$1, CON2.P$5, CON3.P$4, U$1.GND1, U$1.GND2, U$1.GND3, U$1.GND4, U$1.GND6, U$1.GND7, U$1.GND8; no longer IM.GND, R4.1
- net GPSRX: now also CON1.P$3; no longer U$2.RXD
- net GPSTX: now also CON1.P$4; no longer U$2.TXD
- net IM_BUSY: now also CON2.P$3; no longer IM.BUSY/IO1
- net IM_RESET: now also CON2.P$4; no longer IM.RESET
- net IM_RX: now also CON2.P$2; no longer IM.RXD/IO6
- net IM_TX: now also CON2.P$1; no longer IM.TXD/IO7
- net SCK: no longer CN1.CLK, R10.2, R6.2
- net SCL: now also CAM.1
- net SDA: now also CAM.2
Other:
- note added: "ECHO"
- moved on the sheet: BMP1, BMX2, CAM, CN1, MD0, MOS1, MOS2, PIXY2, POW, R1, R10, R5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
