File: NSE2023/EAGLE/project/STM32F3logbord/STM32F3logbord.sch (EAGLE design)
At the start: 32 parts, among them CN1 DM3AT, SW1 SRIDE_SWITCH

Commit message: a
a
Parts:
- removed CON1: (no value), XR Connector:2PIN_SIDE
- removed L1, L2: (no value), Chip LED:OSXX1608C1A
- removed MOS3, MOS4, MOS5: (no value), Chip MOSFET:PCH_SSM6J808R
- removed R13: 100k, rcl:R-US_R0603
- removed U$3: STLINK, STLink:STLINK
- added BOOT: (no value), pinhead:PINHD-1X2/90
- added C3: 4.7uF, rcl:C-USC1608
- added C4: 10nF, rcl:C-USC1608
- added C5: 0.1uF, rcl:C-USC1608
- added C6, C7: 30pF, rcl:C-USC1608
- added CHOICEMOS1, CHOICEMOS2, SWITCHMOS: (no value), Chip MOSFET:PCH_SSM6J808R
- added CRY1: (no value), Crystal:8MHZ
- added LED0, LED1, PWR: (no value), Chip LED:OSXX1608C1A
- added POWER, SIGNAL: (no value), XR Connector:4PIN_SIDE
- added R11: DNF, rcl:R-US_R0603
- added R16: 100, rcl:R-US_R0603
- added R17, R18, R19, R9: 10k, rcl:R-US_R0603
- added RST: (no value), Tact switch:TVAF06-A020B-R
- added STLINK1: (no value), pinhead:PINHD-1X5/90
- added SWITCHRES: 100k, rcl:R-US_R0603
- C1, C2: value (none) -> 100nF; device rcl:C-USC3216 -> rcl:C-USC1608
- R1: value 10k -> 10k or DNF; device rcl:R-EU_R0603 -> rcl:R-US_R0603
- R10: value 10 -> 100; device rcl:R-US_R2512 -> rcl:R-US_R0603
- R2: device rcl:R-EU_R0603 -> rcl:R-US_R0603
Connections:
- removed net BATTEOUT: MOS3.1, MOS3.2, MOS3.5, MOS3.6, U$6.OUT+
- removed net N$15: MOS5.3, R13.1, SW1.L
- new net BIT1: R18.1, SIGNAL.P$3, U$1.PA12/CAN_TX
- new net BIT2: R19.1, SIGNAL.P$4, U$1.PA11/CAN_RX
- new net BOOT0: BOOT.2, R2.1, U$1.BOOT0
- new net MAINBATTE: CHOICEMOS1.1, CHOICEMOS1.2, CHOICEMOS1.5, CHOICEMOS1.6, U$6.OUT+
- new net N$7: C7.1, CRY1.P$2, R11.1
- new net N$8: POWER.P$1
- new net N$9: R18.2, R19.2
- new net NRST: C5.1, R1.1, RST.P$1
- new net OSC_IN: C6.1, CRY1.P$1, U$1.PF0
- new net OSC_OUT: R11.2, U$1.PF1
- new net SWITCH: POWER.P$3, SW1.L, SWITCHMOS.3, SWITCHRES.1
- net +3V3: now also BOOT.1, C1.1, C3.1, C4.1, PWR.AN, R17.2, R9.2, STLINK1.5; no longer U$3.3V3
- net FPLOW: now also CHOICEMOS1.3, CHOICEMOS2.1, CHOICEMOS2.2, CHOICEMOS2.3, CHOICEMOS2.5, CHOICEMOS2.6, POWER.P$2, SWITCHMOS.4, SWITCHRES.2; no longer CON1.P$1, MOS3.3, MOS4.1, MOS4.2, MOS4.3, MOS4.5, MOS4.6, MOS5.4, R13.2
- net GND: now also C3.2, C4.2, C5.2, C6.2, C7.2, POWER.P$4, R16.1, R2.2, R3.1, R4.1, RST.P$2, STLINK1.4; no longer CON1.P$2, R2.1, R3.2, R4.2, U$3.GND
- net LED0: now also LED0.AN; no longer L1.AN
- net LED1: now also LED1.AN; no longer L2.AN
- net N$1: no longer C1.1, R1.1
- net N$10: now also CHOICEMOS1.4, CHOICEMOS2.4; no longer MOS3.4, MOS4.4
- net N$11: now also SWITCHMOS.1, SWITCHMOS.2, SWITCHMOS.5, SWITCHMOS.6; no longer MOS5.1, MOS5.2, MOS5.5, MOS5.6
- net N$2: now also PWR.CT, R16.2; no longer R2.2, U$1.BOOT0
- net N$3: now also LED0.CT, R3.2; no longer L1.CT, R3.1
- net N$4: now also LED1.CT, R4.2; no longer L2.CT, R4.1
- net SCL: now also R9.1, SIGNAL.P$1
- net SDA: now also R17.1, SIGNAL.P$2
- net SWCLK: now also STLINK1.3; no longer U$3.SWCLK
- net SWDIO: now also STLINK1.2; no longer U$3.SWDIO
- net SWO: now also STLINK1.1; no longer U$3.SWO
Other:
- note added: "PWR Check"
- note added: "near VDD"
- note added: "near VDD2"
- note added: "near VDDA"
- moved on the sheet: BMX2, C1, C2, CON2, L4, R10, R12, R14, R15, R3, R4, SW1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

Commit message: kato update logbord
Parts:
- removed STLINK1: (no value), pinhead:PINHD-1X5/90
- added STLINK: (no value), pinhead:PINHD-1X5/90
Connections:
- net +3V3: now also STLINK.5; no longer STLINK1.5
- net GND: now also STLINK.4; no longer STLINK1.4
- net SWCLK: now also STLINK.3; no longer STLINK1.3
- net SWDIO: now also STLINK.2; no longer STLINK1.2
- net SWO: now also STLINK.1; no longer STLINK1.1
Changed lines of the file:
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@@
 <part name="+3V14" library="supply1" library_urn="urn:adsk.eagle:library:371" deviceset="+3V3" device=""/>
 <part name="GND17" library="supply1" library_urn="urn:adsk.eagle:library:371" deviceset="GND" device=""/>
-<part name="STLINK1" library="pinhead" library_urn="urn:adsk.eagle:library:325" deviceset="PINHD-1X5" device="/90" package3d_urn="urn:adsk.eagle:package:22467/2"/>
+<part name="STLINK" library="pinhead" library_urn="urn:adsk.eagle:library:325" deviceset="PINHD-1X5" device="/90" package3d_urn="urn:adsk.eagle:package:22467/2"/>
 </parts>
 <sheets>
@@
 <attribute name="VALUE" x="200.66" y="50.8" size="1.778" layer="96"/>
 </instance>
-<instance part="STLINK1" gate="A" x="213.36" y="66.04" smashed="yes">
-<attribute name="NAME" x="207.01" y="74.295" size="1.778" layer="95"/>
-<attribute name="VALUE" x="207.01" y="55.88" size="1.778" layer="96"/>
+<instance part="STLINK" gate="A" x="220.98" y="66.04" smashed="yes">
+<attribute name="NAME" x="214.63" y="74.295" size="1.778" layer="95"/>
+<attribute name="VALUE" x="214.63" y="55.88" size="1.778" layer="96"/>
 </instance>
 </instances>
@@
 </segment>
 <segment>
-<wire x1="142.24" y1="5.08" x2="142.24" y2="17.78" width="0.1524" layer="91"/>
-<pinref part="+3V13" gate="G$1" pin="+3V3"/>
-</segment>
-<segment>
 <pinref part="R9" gate="G$1" pin="2"/>
 <wire x1="137.16" y1="30.48" x2="142.24" y2="30.48" width="0.1524" layer="91"/>
@@
 </segment>
 <segment>
-<wire x1="210.82" y1="60.96" x2="193.04" y2="60.96" width="0.1524" layer="91"/>
+<wire x1="218.44" y1="60.96" x2="193.04" y2="60.96" width="0.1524" layer="91"/>
 <wire x1="193.04" y1="60.96" x2="193.04" y2="73.66" width="0.1524" layer="91"/>
 <pinref part="+3V14" gate="G$1" pin="+3V3"/>
-<pinref part="STLINK1" gate="A" pin="5"/>
+<pinref part="STLINK" gate="A" pin="5"/>
 </segment>
 </net>
@@
 </segment>
 <segment>
-<wire x1="210.82" y1="63.5" x2="203.2" y2="63.5" width="0.1524" layer="91"/>
 <wire x1="203.2" y1="63.5" x2="203.2" y2="55.88" width="0.1524" layer="91"/>
 <pinref part="GND17" gate="1" pin="GND"/>
-<pinref part="STLINK1" gate="A" pin="4"/>
+<pinref part="STLINK" gate="A" pin="4"/>
+<wire x1="218.44" y1="63.5" x2="203.2" y2="63.5" width="0.1524" layer="91"/>
 </segment>
 </net>
@@
 </segment>
 <segment>
-<wire x1="210.82" y1="71.12" x2="205.74" y2="71.12" width="0.1524" layer="91"/>
 <label x="205.74" y="71.12" size="1.778" layer="95" rot="R180" xref="yes"/>
-<pinref part="STLINK1" gate="A" pin="1"/>
+<pinref part="STLINK" gate="A" pin="1"/>
+<wire x1="218.44" y1="71.12" x2="205.74" y2="71.12" width="0.1524" layer="91"/>
 </segment>
 </net>
@@
 </segment>
 <segment>
-<wire x1="210.82" y1="66.04" x2="205.74" y2="66.04" width="0.1524" layer="91"/>
 <label x="205.74" y="66.04" size="1.778" layer="95" rot="R180" xref="yes"/>
-<pinref part="STLINK1" gate="A" pin="3"/>
+<pinref part="STLINK" gate="A" pin="3"/>
+<wire x1="218.44" y1="66.04" x2="205.74" y2="66.04" width="0.1524" layer="91"/>
 </segment>
 </net>
@@
 </segment>
 <segment>
-<wire x1="210.82" y1="68.58" x2="205.74" y2="68.58" width="0.1524" layer="91"/>
 <label x="205.74" y="68.58" size="1.778" layer="95" rot="R180" xref="yes"/>
-<pinref part="STLINK1" gate="A" pin="2"/>
+<pinref part="STLINK" gate="A" pin="2"/>
+<wire x1="218.44" y1="68.58" x2="205.74" y2="68.58" width="0.1524" layer="91"/>
 </segment>
 </net>
@@
 <wire x1="142.24" y1="12.7" x2="142.24" y2="17.78" width="0.1524" layer="91"/>
 <junction x="142.24" y="12.7"/>
-</segment>
-</net>
+<wire x1="142.24" y1="5.08" x2="142.24" y2="17.78" width="0.1524" layer="91"/>
+<pinref part="+3V13" gate="G$1" pin="+3V3"/>
+</segment>
+</net>

Commit message: add
Parts:
- added U$3: F.T.E.LOGO, logo:F.T.E.LOGO
Connections:
- removed net N$8: POWER.P$1
- removed net N$9: R18.2, R19.2
- net +3V3: now also POWER.P$1, R18.2, R19.2
Changed lines of the file:
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@@
 <layer number="97" name="Info" color="7" fill="1" visible="yes" active="yes"/>
 <layer number="98" name="Guide" color="6" fill="1" visible="yes" active="yes"/>
+<layer number="99" name="SpiceOrder" color="5" fill="1" visible="yes" active="yes"/>
+<layer number="200" name="200bmp" color="1" fill="10" visible="yes" active="yes"/>
 </layers>
 <schematic xreflabel="%F%N/%S.%C%R" xrefpart="/%S.%C%R">
@@
 <part name="SIGNAL" library="XR Connector" library_urn="urn:adsk.eagle:library:38467597" deviceset="4PIN_SIDE" device="" package3d_urn="urn:adsk.eagle:package:38473897/3"/>
 <part name="GND5" library="supply1" library_urn="urn:adsk.eagle:library:371" deviceset="GND" device=""/>
-<part name="+3V11" library="supply1" library_urn="urn:adsk.eagle:library:371" deviceset="+3V3" device=""/>
 <part name="R9" library="rcl" library_urn="urn:adsk.eagle:library:334" deviceset="R-US_" device="R0603" package3d_urn="urn:adsk.eagle:package:23555/3" value="10k"/>
 <part name="R17" library="rcl" library_urn="urn:adsk.eagle:library:334" deviceset="R-US_" device="R0603" package3d_urn="urn:adsk.eagle:package:23555/3" value="10k"/>
 <part name="R18" library="rcl" library_urn="urn:adsk.eagle:library:334" deviceset="R-US_" device="R0603" package3d_urn="urn:adsk.eagle:package:23555/3" value="10k"/>
 <part name="R19" library="rcl" library_urn="urn:adsk.eagle:library:334" deviceset="R-US_" device="R0603" package3d_urn="urn:adsk.eagle:package:23555/3" value="10k"/>
-<part name="+3V13" library="supply1" library_urn="urn:adsk.eagle:library:371" deviceset="+3V3" device=""/>
 <part name="+3V12" library="supply1" library_urn="urn:adsk.eagle:library:371" deviceset="+3V3" device=""/>
 <part name="POWER" library="XR Connector" library_urn="urn:adsk.eagle:library:38467597" deviceset="4PIN_SIDE" device="" package3d_urn="urn:adsk.eagle:package:38473897/3"/>
@@
 <part name="GND17" library="supply1" library_urn="urn:adsk.eagle:library:371" deviceset="GND" device=""/>
 <part name="STLINK" library="pinhead" library_urn="urn:adsk.eagle:library:325" deviceset="PINHD-1X5" device="/90" package3d_urn="urn:adsk.eagle:package:22467/2"/>
+<part name="LOGO1" library="logo" library_urn="urn:adsk.eagle:library:264" deviceset="EAGLE-CS-LOGO-43" device=""/>
+<part name="U$3" library="logo" deviceset="F.T.E.LOGO" device=""/>
+<part name="+3V9" library="supply1" library_urn="urn:adsk.eagle:library:371" deviceset="+3V3" device=""/>
+<part name="+3V11" library="supply1" library_urn="urn:adsk.eagle:library:371" deviceset="+3V3" device=""/>
 </parts>
 <sheets>
@@
 <attribute name="VALUE" x="170.18" y="-50.8" size="1.778" layer="96"/>
 </instance>
-<instance part="+3V11" gate="G$1" x="147.32" y="-25.4" smashed="yes">
-<attribute name="VALUE" x="144.78" y="-30.48" size="1.778" layer="96" rot="R90"/>
-</instance>
 <instance part="R9" gate="G$1" x="132.08" y="30.48" smashed="yes">
 <attribute name="NAME" x="128.27" y="31.9786" size="1.778" layer="95"/>
@@
 <attribute name="VALUE" x="128.27" y="1.778" size="1.778" layer="96"/>
 </instance>
-<instance part="+3V13" gate="G$1" x="142.24" y="20.32" smashed="yes">
-<attribute name="VALUE" x="139.7" y="15.24" size="1.778" layer="96" rot="R90"/>
-</instance>
 <instance part="+3V12" gate="G$1" x="142.24" y="38.1" smashed="yes">
 <attribute name="VALUE" x="139.7" y="33.02" size="1.778" layer="96" rot="R90"/>
@@
 <attribute name="NAME" x="214.63" y="74.295" size="1.778" layer="95"/>
 <attribute name="VALUE" x="214.63" y="55.88" size="1.778" layer="96"/>
+</instance>
+<instance part="LOGO1" gate="G$1" x="-86.36" y="-104.14" smashed="yes"/>
+<instance part="U$3" gate="G$1" x="-15.24" y="-81.28" smashed="yes">
+<attribute name="NAME" x="-15.24" y="-91.44" size="1.778" layer="95"/>
+</instance>
+<instance part="+3V9" gate="G$1" x="147.32" y="-22.86" smashed="yes">
+<attribute name="VALUE" x="144.78" y="-27.94" size="1.778" layer="96" rot="R90"/>
+</instance>
+<instance part="+3V11" gate="G$1" x="142.24" y="20.32" smashed="yes">
+<attribute name="VALUE" x="139.7" y="15.24" size="1.778" layer="96" rot="R90"/>
 </instance>
 </instances>
@@
 <pinref part="+3V14" gate="G$1" pin="+3V3"/>
 <pinref part="STLINK" gate="A" pin="5"/>
+</segment>
+<segment>
+<pinref part="POWER" gate="G$1" pin="P$1"/>
+<wire x1="167.64" y1="-27.94" x2="167.64" y2="-33.02" width="0.1524" layer="91"/>
+<wire x1="167.64" y1="-33.02" x2="147.32" y2="-33.02" width="0.1524" layer="91"/>
+<wire x1="147.32" y1="-33.02" x2="147.32" y2="-25.4" width="0.1524" layer="91"/>
+<pinref part="+3V9" gate="G$1" pin="+3V3"/>
+</segment>
+<segment>
+<pinref part="R18" gate="G$1" pin="2"/>
+<wire x1="137.16" y1="12.7" x2="142.24" y2="12.7" width="0.1524" layer="91"/>
+<wire x1="142.24" y1="12.7" x2="142.24" y2="5.08" width="0.1524" layer="91"/>
+<pinref part="R19" gate="G$1" pin="2"/>
+<wire x1="137.16" y1="5.08" x2="142.24" y2="5.08" width="0.1524" layer="91"/>
+<wire x1="142.24" y1="12.7" x2="142.24" y2="17.78" width="0.1524" layer="91"/>
+<junction x="142.24" y="12.7"/>
+<pinref part="+3V11" gate="G$1" pin="+3V3"/>
 </segment>
 </net>
@@
 </segment>
 </net>
-<net name="N$8" class="0">
-<segment>
-<wire x1="167.64" y1="-27.94" x2="167.64" y2="-33.02" width="0.1524" layer="91"/>
-<wire x1="167.64" y1="-33.02" x2="147.32" y2="-33.02" width="0.1524" layer="91"/>
-<wire x1="147.32" y1="-33.02" x2="147.32" y2="-27.94" width="0.1524" layer="91"/>
-<wire x1="147.32" y1="-30.48" x2="147.32" y2="-27.94" width="0.1524" layer="91"/>
-<pinref part="+3V11" gate="G$1" pin="+3V3"/>
-<pinref part="POWER" gate="G$1" pin="P$1"/>
-</segment>
-</net>
 <net name="BIT1" class="0">
 <segment>
@@
 </segment>
 </net>
-<net name="N$9" class="0">
-<segment>
-<pinref part="R18" gate="G$1" pin="2"/>
-<wire x1="137.16" y1="12.7" x2="142.24" y2="12.7" width="0.1524" layer="91"/>
-<wire x1="142.24" y1="12.7" x2="142.24" y2="5.08" width="0.1524" layer="91"/>
-<pinref part="R19" gate="G$1" pin="2"/>
-<wire x1="137.16" y1="5.08" x2="142.24" y2="5.08" width="0.1524" layer="91"/>
-<wire x1="142.24" y1="12.7" x2="142.24" y2="17.78" width="0.1524" layer="91"/>
-<junction x="142.24" y="12.7"/>
-<wire x1="142.24" y1="5.08" x2="142.24" y2="17.78" width="0.1524" layer="91"/>
-<pinref part="+3V13" gate="G$1" pin="+3V3"/>
-</segment>
-</net>
