File: NSE2023/EAGLE/project/STM32F3logbord/STM32F3logbord.brd (EAGLE design)
At the start: 60 x 30 mm, 32 parts, among them CN1 DM3AT, SW1 SRIDE_SWITCH

Commit message: kato_logbord
Parts:
- moved R14 94.3 mm to (51.1, 22.7), flipped to the bottom
- moved MOS5 90.2 mm to (45.7, 8.89), flipped to the bottom
- moved R13 90.0 mm to (36.8, 16.1), turned to 180 degrees
- moved R12 89.7 mm to (55.9, 22.7), flipped to the bottom
- moved U$4 82.6 mm to (59.7, 15.2), flipped to the bottom
- moved R15 78.3 mm to (8.00, 7.11), turned to 270 degrees
- moved L4 75.6 mm to (4.06, 6.86), turned to 270 degrees
- moved MOS3 73.6 mm to (45.7, 20.3), flipped to the bottom
- moved MOS4 73.2 mm to (45.7, 14.6), flipped to the bottom
- moved SW1 63.1 mm to (6.35, 2.54)
- moved U$5 52.6 mm to (36.8, 21.6), turned to 270 degrees
- moved CON2 35.5 mm to (9.78, 13.7), turned to 270 degrees
- moved R3 30.1 mm to (55.9, 18.1), flipped to the bottom, turned to 180 degrees
- moved R4 28.3 mm to (51.0, 18.2), flipped to the bottom, turned to 180 degrees
- moved CON1 27.6 mm to (9.91, 21.8), turned to 270 degrees
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Routing:
- net GND: track 0.00 -> 210.7 mm, vias 0 -> 7
- net +3V3: track 0.00 -> 95.3 mm, vias 0 -> 4
- net FPLOW: track 0.00 -> 84.1 mm, vias 0 -> 5
- net SDA: track 0.00 -> 71.2 mm, vias 0 -> 2
- net N$11: track 0.00 -> 63.3 mm, vias 0 -> 1
- net SCL: track 0.00 -> 58.6 mm, vias 0 -> 2
- net SWCLK: track 0.00 -> 55.8 mm, vias 0 -> 4
- net N$15: track 0.00 -> 52.8 mm, vias 0 -> 5
- net N$12: track 0.00 -> 50.7 mm, vias 0 -> 2
- net N$13: track 0.00 -> 47.6 mm
- net SWDIO: track 0.00 -> 40.7 mm, vias 0 -> 3
- net SWO: track 0.00 -> 35.4 mm, vias 0 -> 2
- net N$3: track 0.00 -> 33.2 mm, vias 0 -> 1
- net N$1: track 0.00 -> 31.1 mm, vias 0 -> 2
- net N$5: track 0.00 -> 29.6 mm, vias 0 -> 1
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
Commit message: a
a
Parts:
- removed CON1: (no value), XR Connector:2PIN_SIDE
- removed L1, L2: (no value), Chip LED:OSXX1608C1A
- removed MOS3, MOS4, MOS5: (no value), Chip MOSFET:SSM6J808R
- removed R13: 100k, rcl:R0603
- removed U$3: STLINK, STLink:STLINK
- added BOOT: (no value), pinhead:1X02/90
- added C3: 4.7uF, rcl:C1608
- added C4: 10nF, rcl:C1608
- added C5: 0.1uF, rcl:C1608
- added C6, C7: 30pF, rcl:C1608
- added CHOICEMOS1, CHOICEMOS2, SWITCHMOS: (no value), Chip MOSFET:SSM6J808R
- added CRY1: (no value), Crystal:CRYSTAL
- added LED0, LED1, PWR: (no value), Chip LED:OSXX1608C1A
- added POWER, SIGNAL: (no value), XR Connector:4PIN_SIDE
- added R11: DNF, rcl:R0603
- added R16: 100, rcl:R0603
- added R17, R18, R19, R9: 10k, rcl:R0603
- added RST: (no value), Tact switch:TVAF06-A020B-R
- added STLINK1: (no value), pinhead:1X05/90
- added SWITCHRES: 100k, rcl:R0603
- C1, C2: value (none) -> 100nF; device rcl:C3216 -> rcl:C1608
- R1: value 10k -> 10k or DNF
- R10: value 10 -> 100; device rcl:R2512 -> rcl:R0603
- moved R14 52.4 mm to (2.54, 2.92), turned to 270 degrees
- moved R12 51.7 mm to (6.35, 7.75), turned to 180 degrees
- moved U$6 43.1 mm to (15.7, 36.7), flipped to the bottom
- moved R15 29.0 mm to (37.0, 6.35), flipped to the bottom, turned to 180 degrees
- moved R8 28.8 mm to (43.9, 27.0), turned to 180 degrees
- moved SW1 27.3 mm to (2.67, 29.6), turned to 90 degrees
- moved R10 26.9 mm to (40.9, 19.6), flipped to the top
- moved R1 25.3 mm to (45.7, 34.3), turned to 180 degrees
- moved R6 24.3 mm to (43.9, 22.3), turned to 180 degrees
- moved R2 22.2 mm to (29.2, 6.35), flipped to the bottom, turned to 270 degrees
- moved U$1 22.1 mm to (43.3, 16.9), turned to 180 degrees
- moved R5 20.8 mm to (43.9, 20.1), turned to 180 degrees
- moved R7 19.7 mm to (43.9, 24.5), turned to 180 degrees
- moved U$5 19.3 mm to (44.7, 3.94)
- moved CN1 18.2 mm to (40.1, 29.1)
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Connections:
- removed net BATTEOUT: MOS3.1, MOS3.2, MOS3.5, MOS3.6, U$6.V+
- removed net N$15: MOS5.3, R13.1, SW1.L
- new net BIT1: R18.1, SIGNAL.P$3, U$1.PA12/CAN_TX
- new net BIT2: R19.1, SIGNAL.P$4, U$1.PA11/CAN_RX
- new net BOOT0: BOOT.2, R2.1, U$1.BOOT
- new net MAINBATTE: CHOICEMOS1.1, CHOICEMOS1.2, CHOICEMOS1.5, CHOICEMOS1.6, U$6.V+
- new net N$7: C7.1, CRY1.P$2, R11.1
- new net N$8: POWER.P$1
- new net N$9: R18.2, R19.2
- new net NRST: C5.1, R1.1, RST.P$1
- new net OSC_IN: C6.1, CRY1.P$1, U$1.PF0
- new net OSC_OUT: R11.2, U$1.PF1
- new net SWITCH: POWER.P$3, SW1.L, SWITCHMOS.3, SWITCHRES.1
- net +3V3: now also BOOT.1, C1.1, C3.1, C4.1, PWR.AN, R17.2, R9.2, STLINK1.5; no longer U$3.3V3
- net FPLOW: now also CHOICEMOS1.3, CHOICEMOS2.1, CHOICEMOS2.2, CHOICEMOS2.3, CHOICEMOS2.5, CHOICEMOS2.6, POWER.P$2, SWITCHMOS.4, SWITCHRES.2; no longer CON1.P$1, MOS3.3, MOS4.1, MOS4.2, MOS4.3, MOS4.5, MOS4.6, MOS5.4, R13.2
- net GND: now also C3.2, C4.2, C5.2, C6.2, C7.2, POWER.P$4, R16.1, R2.2, R3.1, R4.1, RST.P$2, STLINK1.4; no longer CON1.P$2, R2.1, R3.2, R4.2, U$3.GND
- net LED0: now also LED0.AN; no longer L1.AN
- net LED1: now also LED1.AN; no longer L2.AN
- net N$1: no longer C1.1, R1.1
- net N$10: now also CHOICEMOS1.4, CHOICEMOS2.4; no longer MOS3.4, MOS4.4
- net N$11: now also SWITCHMOS.1, SWITCHMOS.2, SWITCHMOS.5, SWITCHMOS.6; no longer MOS5.1, MOS5.2, MOS5.5, MOS5.6
- net N$2: now also PWR.CT, R16.2; no longer R2.2, U$1.BOOT
- net N$3: now also LED0.CT, R3.2; no longer L1.CT, R3.1
- net N$4: now also LED1.CT, R4.2; no longer L2.CT, R4.1
- net SCL: now also R9.1, SIGNAL.P$1
- net SDA: now also R17.1, SIGNAL.P$2
- net SWCLK: now also STLINK1.3; no longer U$3.SWCLK
- net SWDIO: now also STLINK1.2; no longer U$3.SWDIO
- net SWO: now also STLINK1.1; no longer U$3.SWO
Routing:
- net GND: track 210.7 -> 0.00 mm, vias 7 -> 0
- net +3V3: track 95.3 -> 0.00 mm, vias 4 -> 0
- net FPLOW: track 84.1 -> 0.00 mm, vias 5 -> 0
- net SDA: track 71.2 -> 0.00 mm, vias 2 -> 0
- net N$11: track 63.3 -> 0.00 mm, vias 1 -> 0
- net SCL: track 58.6 -> 0.00 mm, vias 2 -> 0
- net SWCLK: track 55.8 -> 0.00 mm, vias 4 -> 0
- net N$15: track 52.8 -> 0.00 mm, vias 5 -> 0
- net N$12: track 50.7 -> 0.00 mm, vias 2 -> 0
- net N$13: track 47.6 -> 0.00 mm
- net SWDIO: track 40.7 -> 0.00 mm, vias 3 -> 0
- net SWO: track 35.4 -> 0.00 mm, vias 2 -> 0
- net N$3: track 33.2 -> 0.00 mm, vias 1 -> 0
- net N$1: track 31.1 -> 0.00 mm, vias 2 -> 0
- net N$5: track 29.6 -> 0.00 mm, vias 1 -> 0
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Other:
- board size 60 x 30 mm -> 50 x 40 mm

Commit message: add
Parts:
- moved STLINK1 70.5 mm to (7.24, 40.0)
Routing:
- net GND: track 0.00 -> 222.6 mm, vias 0 -> 3
- net +3V3: track 0.00 -> 194.8 mm, vias 0 -> 3
- net FPLOW: track 0.00 -> 116.5 mm, vias 0 -> 5
- net SDA: track 0.00 -> 109.1 mm, vias 0 -> 1
- net BIT1: track 0.00 -> 68.3 mm, vias 0 -> 2
- net N$11: track 0.00 -> 64.9 mm, vias 0 -> 1
- net SCL: track 0.00 -> 63.7 mm, vias 0 -> 3
- net N$5: track 0.00 -> 61.2 mm, vias 0 -> 1
- net SWO: track 0.00 -> 55.8 mm, vias 0 -> 2
- net SWCLK: track 0.00 -> 53.9 mm, vias 0 -> 4
- net BIT2: track 0.00 -> 52.9 mm, vias 0 -> 4
- net SWDIO: track 0.00 -> 47.1 mm, vias 0 -> 4
- net N$16: track 0.00 -> 40.2 mm, vias 0 -> 1
- net SWITCH: track 0.00 -> 35.8 mm, vias 0 -> 1
- net OSC_IN: track 0.00 -> 32.8 mm, vias 0 -> 1
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
Commit message: kato update logbord
Parts:
- removed STLINK1: (no value), pinhead:1X05/90
- added STLINK: (no value), pinhead:1X05/90
- moved L4 44.1 mm to (45.0, 36.2), turned to 270 degrees
- moved R14 35.6 mm to (31.1, 24.1), flipped to the top
- moved C6 32.8 mm to (48.3, 10.4), turned to 270 degrees
- moved R11 29.4 mm to (48.3, 14.1), turned to 90 degrees
- moved R12 27.0 mm to (27.8, 24.1), flipped to the top, turned to 90 degrees
- moved BOOT 26.1 mm to (6.22, 10.0), flipped to the bottom
- moved C5 26.1 mm to (27.9, 19.1), turned to 90 degrees
- moved CHOICEMOS1 26.0 mm to (22.7, 24.3), flipped to the top, turned to 270 degrees
- moved RST 24.3 mm to (22.9, 19.1), turned to 180 degrees
- moved C7 24.1 mm to (48.3, 17.8), turned to 90 degrees
- moved CRY1 23.2 mm to (44.8, 15.0), turned to 270 degrees
- moved C4 20.8 mm to (30.5, 3.81), turned to 180 degrees
- moved R2 19.9 mm to (11.4, 15.2)
- moved CHOICEMOS2 15.6 mm to (16.0, 24.3), flipped to the top, turned to 270 degrees
- moved SWITCHMOS 13.3 mm to (16.5, 19.1), flipped to the top
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Connections:
- net +3V3: now also STLINK.5; no longer STLINK1.5
- net GND: now also STLINK.4; no longer STLINK1.4
- net SWCLK: now also STLINK.3; no longer STLINK1.3
- net SWDIO: now also STLINK.2; no longer STLINK1.2
- net SWO: now also STLINK.1; no longer STLINK1.1
Routing:
- net N$11: track 64.9 -> 129.2 mm
- net GND: track 222.6 -> 265.1 mm, vias 3 -> 1
- net SDA: track 109.1 -> 70.4 mm, vias 1 -> 2
- net BOOT0: track 18.8 -> 53.4 mm, vias 1 -> 2
- net NRST: track 8.39 -> 35.7 mm, vias 0 -> 2
- net OSC_IN: track 32.8 -> 8.32 mm, vias 1 -> 0
- net OSC_OUT: track 32.1 -> 8.36 mm, vias 4 -> 0
- net BIT1: track 68.3 -> 44.7 mm
- net FPLOW: track 116.5 -> 94.3 mm, vias 5 -> 3
- net LED0: track 16.6 -> 37.7 mm, vias 0 -> 2
- net SWO: track 55.8 -> 69.0 mm, vias 2 -> 1
- net N$13: track 19.4 -> 28.3 mm, vias 0 -> 1
- net SCL: track 63.7 -> 71.7 mm, vias 3 -> 2
- net SWDIO: track 47.1 -> 39.4 mm, vias 4 -> 2
- net BIT2: track 52.9 -> 45.4 mm, vias 4 -> 1
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
Commit message: add
Parts:
- added U$3: F.T.E.LOGO, logo:LOGO
Connections:
- removed net N$8: POWER.P$1
- removed net N$9: R18.2, R19.2
- net +3V3: now also POWER.P$1, R18.2, R19.2
Routing:
- net N$11: track 129.2 -> 65.8 mm, vias 1 -> 2
- net +3V3: track 198.0 -> 222.0 mm, vias 10 -> 4
- net SWO: track 69.0 -> 52.0 mm
- net LED0: track 37.7 -> 26.2 mm
- net SWDIO: track 39.4 -> 50.2 mm, vias 2 -> 1
- net BOOT0: track 53.4 -> 64.1 mm
- net N$13: track 28.3 -> 20.5 mm
- net BIT1: track 44.7 -> 52.1 mm, vias 2 -> 1
- net GND: track 265.1 -> 271.7 mm, vias 1 -> 3
- net SWCLK: track 48.0 -> 54.4 mm
- net SDA: track 70.4 -> 76.2 mm, vias 2 -> 1
- net FPLOW: track 94.3 -> 89.1 mm, vias 3 -> 4
- net N$9: track 4.99 -> 0.00 mm, vias 2 -> 0
- net N$16: track 41.5 -> 45.2 mm
- net MISO: track 16.8 -> 15.2 mm
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Other:
- board size 50 x 40 mm -> 50 x 50 mm
- board text added: "3V3"
- board text added: "BIT1"
- board text added: "BIT2"
- board text added: "CLK"
- board text added: "DIO"
- board text added: "FP"
- board text added: "GND"
- board text added: "OFF"
- board text added: "SCL"
- board text added: "SDA"
- board text added: "SW"
- board text added: "SWO"

Commit message: add
Routing:
- net +3V3: track 222.0 -> 181.3 mm, vias 4 -> 7
- net N$11: track 65.8 -> 103.8 mm
- net GND: track 271.7 -> 248.1 mm, vias 3 -> 2
- net MAINBATTE: track 18.9 -> 34.6 mm, vias 3 -> 1
- net LED1: track 27.4 -> 41.9 mm
- net SWCLK: track 54.4 -> 44.0 mm, vias 1 -> 3
- net SDA: track 76.2 -> 83.2 mm, vias 1 -> 4
- net BIT1: track 52.1 -> 45.7 mm, vias 1 -> 2
- net BOOT0: track 64.1 -> 58.0 mm, vias 2 -> 1
- net N$5: track 61.5 -> 65.8 mm, vias 1 -> 2
- net N$12: track 16.8 -> 13.4 mm
- net BIT2: track 43.8 -> 47.0 mm
- net N$13: track 20.5 -> 23.7 mm
- net SWO: track 52.0 -> 49.0 mm, vias 1 -> 3
- net SWDIO: track 50.2 -> 47.8 mm, vias 1 -> 2
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