File: NSE2023/EAGLE/project/STM32F3_Motherver_v2/Down Linker ver2.0.0.sch (EAGLE design)
At the start: 27 parts

Commit message: create final board NSE2023
Parts:
- removed BOOT: (no value), pinhead:PINHD-1X2/90
- removed STLINK: (no value), pinhead:PINHD-1X5/90
- added JP1: (no value), pinhead:PINHD-2X10/90
- added U$4: F.T.E.LOGO, logo:F.T.E.LOGO
Connections:
- new net FPRAW: JP1.6, JP3.10
- new net SW: JP1.4, JP3.8
- net +3V3: now also JP1.1, JP1.17, JP1.18, JP1.9; no longer BOOT.1, STLINK.5
- net +5V: now also JP1.8
- net BIT1: no longer JP3.10
- net BIT2: no longer JP3.8
- net BOOT0: now also JP1.10; no longer BOOT.2
- net GND: now also JP1.19, JP1.20, JP1.7; no longer STLINK.4
- net PWM: now also JP1.2
- net SCL: now also JP1.5
- net SDA: now also JP1.3
- net SWCLK: now also JP1.15, JP1.16; no longer STLINK.3
- net SWDIO: now also JP1.13, JP1.14; no longer STLINK.2
- net SWO: now also JP1.11, JP1.12; no longer STLINK.1
Other:
- moved on the sheet: JP3

Commit message: www
Parts:
- removed C6, C7: 30pF, rcl:C-USC1608
- removed CRY1: (no value), Crystal:8MHZ
- removed JP1: (no value), pinhead:PINHD-2X10/90
- removed R4: DNF, rcl:R-US_R0603
- removed U$4: F.T.E.LOGO, logo:F.T.E.LOGO
- added JP2: (no value), pinhead:PINHD-2X6/90
Connections:
- removed net N$3: C7.1, CRY1.P$2, R4.1
- net +3V3: now also JP2.9; no longer JP1.1, JP1.17, JP1.18, JP1.9
- net +5V: now also JP2.2; no longer JP1.8
- net BOOT0: no longer JP1.10
- net FPRAW: now also JP2.12; no longer JP1.6
- net GND: now also JP2.11; no longer C6.2, C7.2, JP1.19, JP1.20, JP1.7
- net NRST: now also JP2.8
- net OSC_IN: no longer C6.1, CRY1.P$1
- net OSC_OUT: no longer R4.2
- net PWM: now also JP2.1; no longer JP1.2
- net SCL: now also JP2.6; no longer JP1.5
- net SDA: now also JP2.4; no longer JP1.3
- net SW: now also JP2.10; no longer JP1.4
- net SWCLK: now also JP2.7; no longer JP1.15, JP1.16
- net SWDIO: now also JP2.5; no longer JP1.13, JP1.14
- net SWO: now also JP2.3; no longer JP1.11, JP1.12
