File: NSE2023/EAGLE/project/STM32F3_Motherver_v2/Logger ver2.0.0.brd (EAGLE design)
At the start: 35 x 45 mm, 24 parts

Commit message: create final board NSE2023
Parts:
- removed BOOT: (no value), pinhead:1X02/90
- removed U$3: F.T.E.LOGO, logo:LOGO
- added CN1: DM3AT, microSD:DM3AT
- added R10, R7, R8, R9: 10k, rcl:R0603
- added R11: 100, rcl:R0603
- added U$4: F.T.E.LOGO, logo:LOGO
- moved C6 25.4 mm to (1.77, 10.8), turned to 270 degrees
- moved R5 22.0 mm to (1.68, 32.1), turned to 270 degrees
- moved LED0 19.7 mm to (3.70, 32.0), turned to 270 degrees
- moved R6 17.2 mm to (5.96, 32.1), turned to 270 degrees
- moved C1 16.1 mm to (3.64, 17.0), turned to 180 degrees
- moved LED1 15.4 mm to (8.08, 32.0), turned to 270 degrees
- moved CRY1 15.2 mm to (8.49, 10.8), turned to 180 degrees
- moved R3 14.1 mm to (10.6, 32.0), turned to 270 degrees
- moved PWR 13.5 mm to (12.5, 32.1), turned to 270 degrees
- moved C7 13.0 mm to (15.6, 10.7), turned to 90 degrees
- moved R1 12.9 mm to (21.2, 10.7), turned to 90 degrees
- moved BMX1 12.4 mm to (14.9, 26.9), flipped to the bottom, turned to 90 degrees
- moved R4 11.4 mm to (7.45, 15.0), turned to 90 degrees
- moved R2 11.1 mm to (13.5, 36.7)
- moved C4 9.47 mm to (9.61, 15.0), turned to 270 degrees
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Connections:
- new net MISO: CN1.DAT0, R10.1, U$1.PA6/SPI1_MISO
- new net MOSI: CN1.CMD, R8.1, U$1.PA7/SPI1_MOSI
- new net N$11: JP3.17, JP3.4
- new net N$7: CN1.CLK, R11.2, R9.1
- new net NSS: CN1.CD/DAT3, R7.1, U$1.PA4/SPI1_NSS
- new net SCK: R11.1, U$1.PA5/SPI1_SCK
- net +3V3: now also CN1.VDD, JP1.9, R10.2, R7.2, R8.2, R9.2; no longer BOOT.1
- net +5V: no longer JP3.17, JP3.4
- net BIT1: now also JP3.10; no longer U$1.PA12/CAN_TX
- net BIT2: now also JP3.8; no longer U$1.PA11/CAN_RX
- net BOOT0: now also JP1.10; no longer BOOT.2
- net FPRAW: no longer JP3.10
- net GND: now also CN1.VSS
- net PWM: no longer U$1.PA5/SPI1_SCK
- net SW: no longer JP3.8
Routing:
- net FPRAW: track 70.2 -> 0.00 mm, vias 2 -> 0
- net +5V: track 69.1 -> 0.00 mm
- net PWM: track 95.3 -> 44.4 mm, vias 2 -> 0
- net SW: track 44.4 -> 0.00 mm
- net BOOT0: track 45.3 -> 89.3 mm, vias 1 -> 0
- net SDA: track 76.8 -> 105.2 mm
- net NRST: track 25.1 -> 49.6 mm
- net BIT1: track 26.1 -> 3.60 mm, vias 2 -> 0
- net FP_CHECKER: track 2.52 -> 22.7 mm
- net N$11: track 0.00 -> 19.9 mm
- net SCL: track 92.8 -> 73.3 mm
- net MISO: track 0.00 -> 15.5 mm, vias 0 -> 2
- net SWDIO: track 43.6 -> 29.1 mm, vias 2 -> 0
- net SWCLK: track 53.2 -> 39.5 mm, vias 2 -> 1
- net NSS: track 0.00 -> 13.6 mm, vias 0 -> 3
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Other:
- board text removed: "3V3"
- board text removed: "CLK"
- board text removed: "DIO"
- board text removed: "GND"

Commit message: www
Parts:
- removed C6, C7: 30pF, rcl:C1608
- removed CRY1: (no value), Crystal:CRYSTAL
- removed R4: DNF, rcl:R0603
- JP1: device pinhead:2X10/90 -> pinhead:2X05/90
- moved U$4 24.8 mm to (1.00, 7.00)
- moved R2 24.5 mm to (17.3, 12.5), turned to 270 degrees
- moved C5 24.3 mm to (20.5, 12.5), turned to 270 degrees
- moved C1 21.7 mm to (25.0, 13.0)
- moved C4 19.6 mm to (28.6, 20.0), flipped to the bottom
- moved U$1 18.0 mm to (30.0, 23.9), turned to 180 degrees
- moved R10 15.7 mm to (27.7, 31.8), turned to 90 degrees
- moved R11 14.9 mm to (27.6, 24.2), turned to 270 degrees
- moved RST 14.4 mm to (18.2, 18.4), turned to 180 degrees
- moved CN1 14.2 mm to (25.8, 34.3), turned to 180 degrees
- moved R9 13.1 mm to (25.7, 31.8), turned to 90 degrees
- moved R8 10.6 mm to (23.6, 31.8), turned to 90 degrees
- moved R7 8.41 mm to (21.6, 31.8), turned to 90 degrees
- moved R1 8.12 mm to (29.0, 13.0), turned to 0 degrees
- moved C2 6.48 mm to (20.1, 23.9), turned to 90 degrees
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Connections:
- removed net +5V: JP1.8
- removed net N$3: C7.1, CRY1.P$2, R4.1
- removed net OSC_IN: C6.1, CRY1.P$1, U$1.PF0
- removed net OSC_OUT: R4.2, U$1.PF1
- net +3V3: now also JP1.7; no longer JP1.1, JP1.17, JP1.18, JP1.9
- net BOOT0: no longer JP1.10
- net FPRAW: now also JP1.10; no longer JP1.6
- net GND: now also JP1.9; no longer C6.2, C7.2, JP1.19, JP1.20, JP1.7
- net NRST: now also JP1.6
- net PWM: no longer JP1.2
- net SCL: now also JP1.4; no longer JP1.5
- net SDA: now also JP1.2; no longer JP1.3
- net SW: now also JP1.8; no longer JP1.4
- net SWCLK: now also JP1.5; no longer JP1.15, JP1.16
- net SWDIO: now also JP1.3; no longer JP1.13, JP1.14
- net SWO: now also JP1.1; no longer JP1.11, JP1.12
Routing:
- net BOOT0: track 89.3 -> 2.49 mm
- net NRST: track 49.6 -> 98.8 mm, vias 0 -> 2
- net PWM: track 44.4 -> 0.00 mm
- net SDA: track 105.2 -> 73.9 mm, vias 2 -> 1
- net GND: track 186.3 -> 157.4 mm
- net OSC_IN: track 13.5 -> 0.00 mm, vias 2 -> 0
- net N$3: track 10.0 -> 0.00 mm
- net SWDIO: track 29.1 -> 37.3 mm, vias 0 -> 2
- net SWO: track 50.6 -> 43.1 mm
- net MISO: track 15.5 -> 8.65 mm, vias 2 -> 1
- net LED0: track 18.6 -> 24.7 mm
- net LOGTX: track 27.1 -> 21.8 mm, vias 3 -> 0
- net LED1: track 11.7 -> 16.9 mm
- net FP_CHECKER: track 22.7 -> 17.6 mm, vias 0 -> 1
- net SCL: track 73.3 -> 78.0 mm, vias 3 -> 1
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
Commit message: create final board
Parts:
- moved BMX1 9.49 mm to (4.12, 27.9), flipped to the top
- moved U$4 4.00 mm to (1.00, 3.00)
- moved C4 3.65 mm to (28.0, 16.4), turned to 0 degrees
- moved C1 2.00 mm to (25.0, 11.0)
- moved R1 2.00 mm to (29.0, 11.0)
- moved U$1 2.00 mm to (30.0, 21.9)
- moved R10 0.79 mm to (28.5, 31.8)
- moved R11 0.68 mm to (27.4, 24.8), flipped to the top, turned to 90 degrees
- moved R7 0.61 mm to (21.0, 31.8)
- moved R9 0.32 mm to (26.0, 31.8)
- moved R8 0.15 mm to (23.5, 31.8)
Connections:
- net BIT1: no longer JP3.10
- net BIT2: no longer JP3.8
- net FPRAW: now also JP3.10
- net SW: now also JP3.8
Routing:
- net SW: track 0.00 -> 52.5 mm, vias 0 -> 2
- net FPRAW: track 0.00 -> 49.2 mm
- net SWO: track 43.1 -> 70.4 mm, vias 1 -> 2
- net +3V3: track 166.8 -> 139.9 mm, vias 1 -> 2
- net NSS: track 15.3 -> 37.0 mm
- net GND: track 157.4 -> 144.0 mm, vias 4 -> 3
- net BIT2: track 8.66 -> 0.00 mm
- net SCL: track 78.0 -> 69.7 mm
- net LOGRX: track 33.9 -> 41.8 mm, vias 0 -> 1
- net SWCLK: track 39.0 -> 32.8 mm, vias 2 -> 3
- net MISO: track 8.65 -> 14.7 mm
- net N$7: track 10.8 -> 5.95 mm
- net LOGTX: track 21.8 -> 17.3 mm, vias 0 -> 2
- net FP_CHECKER: track 17.6 -> 21.6 mm, vias 1 -> 0
- net BIT1: track 3.60 -> 0.00 mm
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- added copper zone on layer 1, net GND
- added copper zone on layer 16, net GND
