File: NSE2023/EAGLE/project/STM32F3_Motherver_v2/Mother Board_ver2.0.0.sch (EAGLE design)
At the start: 36 parts, among them SW1 SRIDE_SWITCH

Commit message: www
Connections:
- net FPRAW: now also PS2.P$12, PS3.P$12
- net SW: no longer PS2.P$12, PS3.P$12
Changed lines of the file:
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@@
 </variantdefs>
 <classes>
-<class number="0" name="default" width="0" drill="0">
+<class number="0" name="default" width="0.4064" drill="0">
 </class>
-<class number="1" name="esp" width="0.254" drill="0.127">
+<class number="1" name="esp" width="0.4064" drill="0.127">
 <clearance class="1" value="0.0254"/>
 </class>
@@
 </segment>
 <segment>
+<pinref part="PS2" gate="G$1" pin="P$14"/>
+<wire x1="7.62" y1="-7.62" x2="12.7" y2="-7.62" width="0.1524" layer="91"/>
+<label x="12.7" y="-7.62" size="1.778" layer="95" xref="yes"/>
+</segment>
+<segment>
+<pinref part="PS1" gate="G$1" pin="P$14"/>
+<wire x1="7.62" y1="38.1" x2="12.7" y2="38.1" width="0.1524" layer="91"/>
+<label x="12.7" y="38.1" size="1.778" layer="95" xref="yes"/>
+</segment>
+</net>
+<net name="FPRAW" class="0">
+<segment>
+<pinref part="PS1" gate="G$1" pin="P$12"/>
+<wire x1="7.62" y1="40.64" x2="12.7" y2="40.64" width="0.1524" layer="91"/>
+<label x="12.7" y="40.64" size="1.778" layer="95" xref="yes"/>
+</segment>
+<segment>
 <pinref part="PS3" gate="G$1" pin="P$12"/>
 <wire x1="7.62" y1="-48.26" x2="12.7" y2="-48.26" width="0.1524" layer="91"/>
@@
 <label x="12.7" y="-5.08" size="1.778" layer="95" xref="yes"/>
 </segment>
-<segment>
-<pinref part="PS2" gate="G$1" pin="P$14"/>
-<wire x1="7.62" y1="-7.62" x2="12.7" y2="-7.62" width="0.1524" layer="91"/>
-<label x="12.7" y="-7.62" size="1.778" layer="95" xref="yes"/>
-</segment>
-<segment>
-<pinref part="PS1" gate="G$1" pin="P$14"/>
-<wire x1="7.62" y1="38.1" x2="12.7" y2="38.1" width="0.1524" layer="91"/>
-<label x="12.7" y="38.1" size="1.778" layer="95" xref="yes"/>
-</segment>
-</net>
-<net name="FPRAW" class="0">
-<segment>
-<pinref part="PS1" gate="G$1" pin="P$12"/>
-<wire x1="7.62" y1="40.64" x2="12.7" y2="40.64" width="0.1524" layer="91"/>
-<label x="12.7" y="40.64" size="1.778" layer="95" xref="yes"/>
-</segment>
-</net>
+</net>

Commit message: create final board
Parts:
- renumbered PS1 to RC, PS2 to DL, PS3 to GD
