File: NSE2023/EAGLE/project/STM32F3_Motherver_v2/Mother Board_ver2.0.0_under.sch (EAGLE design)
At the start: 6 parts

Commit message: create final board
Parts:
- renumbered CON5 to POWER, CON6 to SENSER-MOTOR, PS1 to DL, PS2 to RC, PS3 to GD
Connections:
- removed net SWCLK0: RC.P$5, RC.P$6
- removed net SWCLK1: DL.P$5, DL.P$6
- removed net SWCLK2: GD.P$5, GD.P$6
- removed net SWDIO0: RC.P$7, RC.P$8
- removed net SWDIO1: DL.P$7, DL.P$8
- removed net SWDIO2: GD.P$7, GD.P$8
- removed net SWO0: RC.P$10, RC.P$9
- removed net SWO1: DL.P$10, DL.P$9
- removed net SWO2: GD.P$10, GD.P$9
- new net NRST0: RC.P$14
- new net NRST1: DL.P$16
- new net NRST2: GD.P$14
- net +3V3: now also DL.P$13, GD.P$17, RC.P$11; no longer DL.P$19, DL.P$3, DL.P$4, GD.P$19, GD.P$3, GD.P$4, RC.P$19, RC.P$3, RC.P$4
- net +5V: now also GD.P$20, RC.P$20; no longer DL.P$14, GD.P$14, RC.P$14
- net FPRAW: now also DL.P$12, GD.P$10, RC.P$10; no longer DL.P$16, GD.P$16, RC.P$16
- net GND: now also DL.P$11, GD.P$9, RC.P$9; no longer DL.P$1, DL.P$13, DL.P$2, GD.P$1, GD.P$13, GD.P$2, RC.P$1, RC.P$13, RC.P$2
- net PWM: now also GD.P$19, RC.P$19; no longer DL.P$20, GD.P$20, RC.P$20
- net SCL0: now also RC.P$16; no longer RC.P$15
- net SCL1: now also DL.P$18; no longer DL.P$15
- net SCL2: now also GD.P$16; no longer GD.P$15
- net SDA0: now also RC.P$18; no longer RC.P$17
- net SDA1: now also DL.P$20; no longer DL.P$17
- net SDA2: now also GD.P$18; no longer GD.P$17
- net SW: now also DL.P$14, GD.P$12, RC.P$12; no longer DL.P$18, GD.P$18, RC.P$18
