File: NSE2023/EAGLE/project/STM32F3logbordv2/STM32F3logbordv2.brd (EAGLE design)
At the start: 50 x 50 mm, 53 parts, among them CN1 DM3AT, SW1 SRIDE_SWITCH

Commit message: create final board
Parts:
- removed BOOT: (no value), pinhead:1X02/90
- removed C6, C7: 30pF, rcl:C1608
- removed CON3, CON4: (no value), XR Connector:2PIN_SIDE
- removed CON5: (no value), XR Connector:3PIN
- removed CRY1: (no value), Crystal:CRYSTAL
- removed R11: DNF, rcl:R0603
- removed R12: 100k, rcl:R0603
- removed R18, R19: 10k, rcl:R0603
- removed U$2: ADXL375, ADXL375:ADXL375
- removed U$7: LT1117-5, LT1117:SOT-223
- added PULLDOWN: 100k, rcl:R0603
- added SIGNAL: (no value), XR Connector:4PIN_SIDE
- R10: value 100 -> 10k
- R6: value 10k -> 100
- moved R14 103.9 mm to (7.00, 25.0), turned to 270 degrees
- moved R13 102.8 mm to (7.00, 29.0), turned to 90 degrees
- moved MOS5 99.6 mm to (12.7, 29.2), turned to 270 degrees
- moved C8 94.6 mm to (13.0, 25.0), turned to 270 degrees
- moved CON1 63.9 mm to (8.89, 34.3), turned to 180 degrees
- moved R2 29.8 mm to (40.7, 9.73), flipped to the top
- moved R15 27.4 mm to (22.5, 25.7), flipped to the bottom, turned to 270 degrees
- moved CHOICEMOS1 26.2 mm to (5.00, 5.00)
- moved R1 24.7 mm to (34.7, 9.73), turned to 90 degrees
- moved L4 23.7 mm to (22.5, 28.7)
- moved U$4 21.8 mm to (30.7, -2.54), flipped to the top, turned to 180 degrees
- moved BMX2 21.3 mm to (15.5, 22.5), turned to 0 degrees
- moved LED1 20.2 mm to (20.0, 28.7)
- moved CHOICEMOS2 19.9 mm to (11.0, 5.00)
- moved R4 19.7 mm to (20.0, 25.7), flipped to the bottom
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Connections:
- removed net +3V2: CON4.P$2
- removed net +5V: CON5.P$2, U$7.2
- removed net BIT1: R18.1, U$1.PA12/CAN_TX
- removed net BIT2: R19.1, U$1.PA11/CAN_RX
- removed net N$5: U$1.PA8
- removed net N$7: C7.1, CRY1.P$2, R11.1
- removed net SCL0: CON2.P$1
- removed net SCL1: CON1.P$1
- removed net SDA0: CON2.P$2
- removed net SDA1: CON1.P$2
- new net N$6: CN1.CLK, R5.1, R6.2
- net +3V3: now also R10.2, R5.2, R7.2, R8.2, SIGNAL.P$3; no longer BOOT.1, R18.2, R19.2, R5.1, R6.1, R7.1, R8.1, U$2.VDDI
- net BOOT0: no longer BOOT.2
- net FPRAW: now also CON1.P$2, PULLDOWN.2; no longer CON3.P$2, R12.2
- net GND: now also CON2.P$1, PULLDOWN.1, SIGNAL.P$4; no longer C6.2, C7.2, CON3.P$1, CON4.P$1, CON5.P$1, U$2.GND1, U$2.GND2, U$7.4
- net MAINBATTE: now also CON2.P$2
- net MISO: now also R10.1; no longer R5.2
- net MOSI: now also R8.1; no longer R7.2
- net N$10: no longer R12.1
- net N$11: no longer U$7.3
- net NSS: now also R7.1; no longer R8.2
- net OSC_IN: no longer C6.1, CRY1.P$1
- net OSC_OUT: no longer R11.2
- net PWM: no longer CON5.P$3
- net SCK: now also R6.1; no longer CN1.CLK, R10.1, R10.2, R6.2
- net SCL: now also SIGNAL.P$1; no longer U$2.SCK
- net SDA: now also SIGNAL.P$2; no longer U$2.SDA
- net SWITCH: now also CON1.P$1
Routing:
- net GND: track 0.00 -> 237.4 mm, vias 0 -> 4
- net +3V3: track 0.00 -> 199.5 mm
- net FPRAW: track 0.00 -> 69.7 mm, vias 0 -> 2
- net FP_CHECKER: track 0.00 -> 68.1 mm, vias 0 -> 2
- net SWO: track 0.00 -> 56.7 mm, vias 0 -> 1
- net SWCLK: track 0.00 -> 55.7 mm, vias 0 -> 3
- net SDA: track 0.00 -> 49.5 mm, vias 0 -> 2
- net SWITCH: track 0.00 -> 48.4 mm, vias 0 -> 1
- net N$11: track 0.00 -> 42.9 mm
- net SCL: track 0.00 -> 39.6 mm, vias 0 -> 1
- net SWDIO: track 0.00 -> 30.4 mm
- net MAINBATTE: track 0.00 -> 25.4 mm
- net LED1: track 0.00 -> 22.2 mm, vias 0 -> 2
- net NSS: track 0.00 -> 18.4 mm, vias 0 -> 2
- net LED0: track 0.00 -> 17.5 mm
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Other:
- board text removed: "FP"
- board text removed: "SW"
