File: NSE2023/EAGLE/project/STM32F3logbordv2/STM32F3logbordv2.sch (EAGLE design)
At the start: 53 parts, among them CN1 DM3AT, SW1 SRIDE_SWITCH

Commit message: create final board
Parts:
- removed BOOT: (no value), pinhead:PINHD-1X2/90
- removed C6, C7: 30pF, rcl:C-USC1608
- removed CON3, CON4: (no value), XR Connector:2PIN_SIDE
- removed CON5: (no value), XR Connector:3PIN
- removed CRY1: (no value), Crystal:8MHZ
- removed R11: DNF, rcl:R-US_R0603
- removed R12: 100k, rcl:R-US_R0603
- removed R18, R19: 10k, rcl:R-US_R0603
- removed U$2: ADXL375, ADXL375:ADXL375
- removed U$7: LT1117-5, LT1117:LT1117-5
- added PULLDOWN: 100k, rcl:R-US_R0603
- added SIGNAL: (no value), XR Connector:4PIN_SIDE
- R10: value 100 -> 10k
- R5, R7, R8: device rcl:R-EU_R0603 -> rcl:R-US_R0603
- R6: value 10k -> 100; device rcl:R-EU_R0603 -> rcl:R-US_R0603
Connections:
- removed net +3V2: CON4.P$2
- removed net +5V: CON5.P$2, U$7.OUT
- removed net BIT1: R18.1, U$1.PA12/CAN_TX
- removed net BIT2: R19.1, U$1.PA11/CAN_RX
- removed net N$5: U$1.PA8
- removed net N$7: C7.1, CRY1.P$2, R11.1
- removed net SCL0: CON2.P$1
- removed net SCL1: CON1.P$1
- removed net SDA0: CON2.P$2
- removed net SDA1: CON1.P$2
- new net N$6: CN1.CLK, R5.1, R6.2
- net +3V3: now also R10.2, R5.2, R7.2, R8.2, SIGNAL.P$3; no longer BOOT.1, R18.2, R19.2, R5.1, R6.1, R7.1, R8.1, U$2.VDDI
- net BOOT0: no longer BOOT.2
- net FPRAW: now also CON1.P$2, PULLDOWN.2; no longer CON3.P$2, R12.2
- net GND: now also CON2.P$1, PULLDOWN.1, SIGNAL.P$4; no longer C6.2, C7.2, CON3.P$1, CON4.P$1, CON5.P$1, U$2.GND1, U$2.GND2, U$7.GND
- net MAINBATTE: now also CON2.P$2
- net MISO: now also R10.1; no longer R5.2
- net MOSI: now also R8.1; no longer R7.2
- net N$10: no longer R12.1
- net N$11: no longer U$7.IN
- net NSS: now also R7.1; no longer R8.2
- net OSC_IN: no longer C6.1, CRY1.P$1
- net OSC_OUT: no longer R11.2
- net PWM: no longer CON5.P$3
- net SCK: now also R6.1; no longer CN1.CLK, R10.1, R10.2, R6.2
- net SCL: now also SIGNAL.P$1; no longer U$2.SCK
- net SDA: now also SIGNAL.P$2; no longer U$2.SDA
- net SWITCH: now also CON1.P$1
Other:
- moved on the sheet: CN1, CON1, CON2, R10
