File: NSE2023/EAGLE/project/STM32F3logbordv2/water ver3.0.0.sch (EAGLE design)
At the start: 11 parts

Commit message: create final board
Parts:
- removed CON3, CON5, CON7: (no value), XR Connector:3PIN
- removed CON4, CON6: (no value), XR Connector:2PIN
- added SIGNAL, SIGNAL1: (no value), XR Connector:4PIN_SIDE
Connections:
- removed net +5V: CON7.P$2
- removed net N$3: CON6.P$2, SRIDE_SWTCH2.L
- removed net N$4: CON6.P$1, SRIDE_SWTCH2.LR
- removed net PWM: CON7.P$3
- new net FPRAW: CON1.P$1, CON2.P$1
- new net SWITCH: CON1.P$2, CON2.P$2, SRIDE_SWTCH2.L
- net +3V3: now also SIGNAL.P$3, SIGNAL1.P$3; no longer CON4.P$1
- net GND: now also SIGNAL.P$4, SIGNAL1.P$4, SRIDE_SWTCH2.LR; no longer CON4.P$2, CON7.P$1
- net SCL0: now also SIGNAL.P$1; no longer CON1.P$2
- net SCL1: now also SIGNAL1.P$1; no longer CON2.P$2
- net SDA0: now also SIGNAL.P$2; no longer CON1.P$1
- net SDA1: now also SIGNAL1.P$2; no longer CON2.P$1
Other:
- moved on the sheet: BMP1, BMP2, CON1, CON2, CON9
